File: CartRiser/CartRiser/CartRiser.kicad_sch (KiCad schematic)
At the start: 6 parts, among them J1 GROM Port, J2 GROM Port

Commit message: trim cart riser
Parts:
- removed H1, H3: MountingHole, MountingHole:MountingHole_3.2mm_M3, symbol Mechanical:MountingHole
Changed lines of the file:
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@@
   (paper "A4")
   (title_block
-    (date "2022-10-16")
-    (rev "V0.5")
+    (date "2022-10-25")
+    (rev "V0.8")
   )
   (junction (at 135.89 26.67) (diameter 0) (color 0 0 0 0)
@@
     (pin "1")
   )
-  (symbol (lib_id "Mechanical:MountingHole") (at 175.26 24.13 0) (unit 1)
-    (in_bom yes) (on_board yes) (fields_autoplaced)
-    (property "Reference" "H1" (id 0) (at 177.8 23.2953 0)
-      (effects (font (size 1.27 1.27)) (justify left))
-    )
-    (property "Value" "MountingHole" (id 1) (at 177.8 25.8322 0)
-      (effects (font (size 1.27 1.27)) (justify left))
-    )
-    (property "Footprint" "MountingHole:MountingHole_3.2mm_M3" (id 2) (at 175.26 24.13 0)
-      (effects (font (size 1.27 1.27)) hide)
-    )
-    (property "Datasheet" "~" (id 3) (at 175.26 24.13 0)
-      (effects (font (size 1.27 1.27)) hide)
-    )
-  )
   (symbol (lib_id "power:+5V") (at 90.17 49.53 90) (unit 1)
     (in_bom yes) (on_board yes) (fields_autoplaced)
@@
     )
     (pin "1")
-  )
-  (symbol (lib_id "Mechanical:MountingHole") (at 175.26 34.29 0) (unit 1)
-    (in_bom yes) (on_board yes) (fields_autoplaced)
-    (property "Reference" "H3" (id 0) (at 177.8 33.4553 0)
-      (effects (font (size 1.27 1.27)) (justify left))
-    )
-    (property "Value" "MountingHole" (id 1) (at 177.8 35.9922 0)
-      (effects (font (size 1.27 1.27)) (justify left))
-    )
-    (property "Footprint" "MountingHole:MountingHole_3.2mm_M3" (id 2) (at 175.26 34.29 0)
-      (effects (font (size 1.27 1.27)) hide)
-    )
-    (property "Datasheet" "~" (id 3) (at 175.26 34.29 0)
-      (effects (font (size 1.27 1.27)) hide)
-    )
   )
   (symbol (lib_id "power:+5V") (at 105.41 121.92 90) (unit 1)
@@
       (reference "#PWR010") (unit 1) (value "GND") (footprint "")
     )
-    (path "/9531e3b7-9ead-4c2b-8c41-d537cec59bca"
-      (reference "H1") (unit 1) (value "MountingHole") (footprint "MountingHole:MountingHole_3.2mm_M3")
-    )
     (path "/861fbb17-591d-457c-9be7-67b5220b8352"
       (reference "H2") (unit 1) (value "MountingHole") (footprint "MountingHole:MountingHole_3.2mm_M3")
     )
-    (path "/b495def4-6f53-46c5-8eb0-a8a672e1e46a"
-      (reference "H3") (unit 1) (value "MountingHole") (footprint "MountingHole:MountingHole_3.2mm_M3")
-    )
     (path "/c4ce91bc-b6af-41ae-ba88-1d7353127ac0"
