File: Keyboard/Keyboard.kicad_pcb (KiCad board)
At the start: 2 copper layers, 282.7 x 108.3 mm, 57 parts, among them J1 computer, SW1 0, SW10 9, SW11 FNCT, SW12 EQUALS, SW14 SLASH, SW16 COLON, SW19 COMMA, SW2 1, SW20 PERIOD, SW23 A, SW24 B, SW25 C, SW26 D, SW27 E, SW28 F, SW29 G, SW3 2, SW30 H, SW31 I, SW32 J, SW33 K, SW34 L, SW35 M, SW36 N, SW37 O, SW38 P, SW39 Q, SW4 3, SW40 R, SW41 S, SW42 T, SW43 U, SW44 V, SW45 W, SW46 X, SW47 Y, SW48 Z, SW49 SHIFT, SW5 4, SW50 spare1, SW6 5, SW61 LOCK, SW64 ENTER, SW65 SPACE, SW69 spare2, SW7 6, SW70 CTRL, SW73 SHIFT, SW8 7, SW9 8

Commit message: unicorn work
Parts:
- removed the SW50 at (283.8, 119.4)
- removed SW69: spare2, Cherry_MX:CHERRY_PCB_100H
- added C1: 0.1µF, Capacitor_THT:C_Disc_D7.0mm_W2.5mm_P5.00mm, F.Cu at (47.0, 138.8)
- added D1: Alpha, LED_THT:LED_D3.0mm, F.Cu at (58.5, 157.7)
- added D2: Power, LED_THT:LED_D3.0mm, F.Cu at (105.0, 107.4)
- added R1: 470Ω, Resistor_THT:R_Axial_DIN0207_L6.3mm_D2.5mm_P7.62mm_Horizontal, F.Cu at (47.8, 149.7)
- added R2: 470Ω, Resistor_THT:R_Axial_DIN0207_L6.3mm_D2.5mm_P7.62mm_Horizontal, F.Cu at (92.4, 107.4)
- added R3: 1KΩ, Resistor_THT:R_Axial_DIN0207_L6.3mm_D2.5mm_P7.62mm_Horizontal, F.Cu at (45.6, 118.5)
- added U1: ATtiny13A-P, Package_DIP:DIP-8_W7.62mm_LongPads, F.Cu at (41.7, 123.9)
- J1: value computer -> Computer; footprint Connector_PinHeader_2.54mm:PinHeader_1x15_P2.54mm_Vertical -> Connector_PinHeader_1.00mm:PinHeader_1x18_P1.00mm_Vertical
- SW44: renamed from SW70; footprint Cherry_MX:CHERRY_PCB_100H -> Button_Switch_Keyboard:SW_Cherry_MX_1.25u_PCB
- SW50: renamed from SW11; footprint Cherry_MX:CHERRY_PCB_100H -> Button_Switch_Keyboard:SW_Cherry_MX_1.25u_PCB
- moved J1 25.6 mm to (73.0, 107.4)
- moved SW31 11.4 mm to (57.2, 167.7), turned to 180 degrees
- moved H1 10.0 mm to (268.0, 203.0)
- moved SW50 7.07 mm to (248.3, 195.7)
- moved SW44 4.98 mm to (105.1, 195.7)
- renumbered H3 to H1, H4 to H2, H5 to H3, H6 to H4, H7 to H5, H8 to H6, SW14 to SW1, SW32 to SW10, SW30 to SW11, SW65 to SW12, SW38 to SW13, SW37 to SW14, SW31 to SW15, SW43 to SW16, SW47 to SW17, SW64 to SW18, SW1 to SW19, SW20 to SW2, SW10 to SW20, SW9 to SW21, SW8 to SW22, SW7 to SW23, SW48 to SW25, SW46 to SW26, SW25 to SW27, SW44 to SW28, SW24 to SW29, SW19 to SW3, SW61 to SW31, SW23 to SW32, SW41 to SW33, SW26 to SW34, SW28 to SW35, SW29 to SW36, SW73 to SW37, SW49 to SW38, SW35 to SW4, SW45 to SW40, SW27 to SW41, SW40 to SW42, SW42 to SW43, SW2 to SW45, SW3 to SW46, SW4 to SW47, SW5 to SW48, SW6 to SW49, SW36 to SW5, SW12 to SW6, SW16 to SW7, SW34 to SW8, SW33 to SW9
Connections:
- SW31 pad 1: PA6 -> VCC
- SW31 pad 2: PB7 -> LOCK
Routing:
- net PB7: track 456.3 -> 249.2 mm
- net PB4: track 308.1 -> 159.8 mm
- net PA3: track 415.8 -> 274.0 mm, vias 1 -> 2
- net VCC: track 0.00 -> 139.8 mm, vias 0 -> 2
- net GND: track 0.00 -> 100.3 mm
- net PB1: track 367.3 -> 268.2 mm, vias 1 -> 0
- net PA5: track 463.8 -> 385.6 mm
- net LOCK: track 0.00 -> 72.2 mm
- net Net-(D1-Pad1): track 0.00 -> 42.8 mm
- net PA6: track 86.5 -> 48.5 mm, vias 0 -> 1
- net PB3: track 207.6 -> 173.9 mm
- net PB0: track 296.2 -> 328.6 mm, vias 1 -> 0
- net PB5: track 329.1 -> 298.9 mm, vias 0 -> 2
- net ~{RESET}: track 0.00 -> 23.9 mm
- net PB2: track 214.4 -> 234.3 mm, vias 0 -> 1
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- added copper zone on B.Cu, net GND
- added copper zone on F.Cu, net GND
Other:
- board text added: "TI99_22 Dan Werner 10/13/2022 V0.8"
- board text removed: "TI99_22 Dan Werner 6/24/2022 V0.5"

Commit message: PCB correction
Parts:
- J1: footprint Connector_PinHeader_1.00mm:PinHeader_1x18_P1.00mm_Vertical -> Connector_PinHeader_2.54mm:PinHeader_1x18_P2.54mm_Vertical
- moved D2 51.9 mm to (156.9, 108.1)
- moved R2 51.9 mm to (144.3, 108.1)
- moved J1 42.3 mm to (115.3, 108.1)
- moved D1 0.10 mm to (58.5, 157.8)
Routing:
- net PB0: track 328.6 -> 260.2 mm
- net PB1: track 268.2 -> 213.6 mm
- net GND: track 100.3 -> 149.5 mm
- net PB3: track 173.9 -> 133.1 mm, vias 0 -> 1
- net PB2: track 234.3 -> 196.5 mm, vias 1 -> 0
- net PA4: track 236.1 -> 203.9 mm, vias 0 -> 1
- net PA3: track 274.0 -> 249.2 mm, vias 2 -> 1
- net PA1: track 306.4 -> 284.2 mm, vias 0 -> 1
- net PA2: track 290.1 -> 269.8 mm, vias 0 -> 1
- net PA6: track 48.5 -> 65.6 mm, vias 1 -> 0
- net ~{RESET}: track 23.9 -> 36.9 mm
- net VCC: track 139.8 -> 151.5 mm, vias 2 -> 0
- net LOCK: track 72.2 -> 60.8 mm
- net PB7: track 249.2 -> 260.3 mm
- net PB4: track 159.8 -> 151.1 mm
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
Commit message: hardware updates
Parts:
- added U2: 74LS125, Package_DIP:DIP-14_W7.62mm_Socket_LongPads, F.Cu at (55.9, 205.2)
- renumbered SW25 to SW24, SW26 to SW25, SW27 to SW26, SW28 to SW27, SW29 to SW28, SW31 to SW29, SW32 to SW30, SW33 to SW31, SW34 to SW32, SW35 to SW33, SW36 to SW34, SW37 to SW35, SW38 to SW36, SW39 to SW37, SW40 to SW38, SW41 to SW39, SW42 to SW40, SW43 to SW41, SW44 to SW42, SW45 to SW43, SW46 to SW44, SW47 to SW45, SW48 to SW46, SW49 to SW47, SW50 to SW48
Connections:
- net Net-(D1-Pad1) renamed ~{LOCKOUT}
- U1 pad 5: PB7 -> unconnected-(U1-Pad5)
- U1 pad 6: PA6 -> unconnected-(U1-Pad6)
Routing:
- net GND: track 149.5 -> 245.1 mm
- net PA6: track 65.6 -> 143.3 mm, vias 0 -> 1
- net PB7: track 260.3 -> 334.9 mm, vias 0 -> 1
- net ~{LOCKOUT}: track 36.0 -> 87.5 mm
- net VCC: track 151.5 -> 196.8 mm
Other:
- board text added: "TI99_22 Dan Werner 11/13/2022 V0.9"
- board text removed: "TI99_22 Dan Werner 10/13/2022 V0.8"
