File: Keyboard/Keyboard.kicad_sch (KiCad schematic)
At the start: 62 parts, among them J1 Computer, SW1 SLASH, SW10 J, SW11 H, SW12 SPACE, SW13 P, SW14 O, SW15 I, SW16 U, SW17 Y, SW18 ENTER, SW19 0, SW2 PERIOD, SW20 9, SW21 8, SW22 7, SW23 6, SW25 Z, SW26 X, SW27 C, SW28 V, SW29 B, SW3 COMMA, SW31 LOCK, SW32 A, SW33 S, SW34 D, SW35 F, SW36 G, SW37 SHIFT, SW38 SHIFT, SW39 Q, SW4 M, SW40 W, SW41 E, SW42 R, SW43 T, SW44 CTRL, SW45 1, SW46 2, SW47 3, SW48 4, SW49 5, SW5 N, SW50 FNCT, SW6 EQUALS, SW7 COLON, SW8 L, SW9 K, U1 ATtiny13A-P

Commit message: PCB correction
Parts:
- J1: footprint Connector_PinHeader_1.00mm:PinHeader_1x18_P1.00mm_Vertical -> Connector_PinHeader_2.54mm:PinHeader_1x18_P2.54mm_Vertical
Changed lines of the file:
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@@
       (effects (font (size 1.27 1.27)) (justify left))
     )
-    (property "Footprint" "Connector_PinHeader_1.00mm:PinHeader_1x18_P1.00mm_Vertical" (id 2) (at 252.73 55.88 0)
+    (property "Footprint" "Connector_PinHeader_2.54mm:PinHeader_1x18_P2.54mm_Vertical" (id 2) (at 252.73 55.88 0)
       (effects (font (size 1.27 1.27)) hide)
     )
@@
     )
     (path "/16537748-b085-4a35-a86b-8164f54e385b"
-      (reference "J1") (unit 1) (value "Computer") (footprint "Connector_PinHeader_1.00mm:PinHeader_1x18_P1.00mm_Vertical")
+      (reference "J1") (unit 1) (value "Computer") (footprint "Connector_PinHeader_2.54mm:PinHeader_1x18_P2.54mm_Vertical")
     )
     (path "/c88be24d-5c7c-404a-9f9c-08aa383122b0"

Commit message: hardware updates
Parts:
- added U2: 74LS125, Package_DIP:DIP-14_W7.62mm_Socket_LongPads, symbol 74xx:74LS125
- renumbered SW25 to SW24, SW26 to SW25, SW27 to SW26, SW28 to SW27, SW29 to SW28, SW31 to SW29, SW32 to SW30, SW33 to SW31, SW34 to SW32, SW35 to SW33, SW36 to SW34, SW37 to SW35, SW38 to SW36, SW39 to SW37, SW40 to SW38, SW41 to SW39, SW42 to SW40, SW43 to SW41, SW44 to SW42, SW45 to SW43, SW46 to SW44, SW47 to SW45, SW48 to SW46, SW49 to SW47, SW50 to SW48
Connections:
- net GND: now also U2.7 (GND)
- net PA6: now also U2.1; no longer U1.6 (PB1)
- net PB7: now also U2.3; no longer U1.5 (PB0)
- net VCC: now also U2.14 (VCC)
- net ~{LOCKOUT}: now reaches D1.1 (K), U1.7 (PB2)
- net ~{LOCKOUT}: now also U2.2
- no-connect marks 1 -> 12
