File: unicornboard/unicorn/unicorn.kicad_pcb (KiCad board)
At the start: 2 copper layers, 100 x 60 mm, 6 parts, among them J1 UNICORN PORT, U1 HV-LV, U2 HV-LV, U3 HV-LV, U4 HV-LV, U5 ESP32_MODULE

Commit message: unicorn work
Parts:
- added H1: MountingHole, MountingHole:MountingHole_3.2mm_M3, F.Cu at (95.5, 96.0)
- added H2: MountingHole, MountingHole:MountingHole_3.2mm_M3, F.Cu at (186.0, 96.0)
- added H3: MountingHole, MountingHole:MountingHole_3.2mm_M3, F.Cu at (95.5, 46.0)
- added H4: MountingHole, MountingHole:MountingHole_3.2mm_M3, F.Cu at (186.0, 46.0)
- J1: footprint Connector_PinHeader_2.54mm:PinHeader_1x15_P2.54mm_Vertical -> Connector_PinHeader_2.54mm:PinHeader_1x16_P2.54mm_Vertical
- moved J1 0.21 mm to (159.4, 47.7)
Connections:
- U5 pad 7: unconnected-(U5-Pad7) -> ~{RESET}
Routing:
- net ~{RESET}: track 0.00 -> 35.2 mm, vias 0 -> 2
- net +5V: track 154.1 -> 155.7 mm
- net ~{GS}: track 45.5 -> 46.9 mm

Commit message: hardware updates
Parts:
- moved U1 2.25 mm to (174.4, 53.0)
- moved U2 2.05 mm to (174.0, 76.3)
- moved U3 0.11 mm to (105.7, 54.3)
- moved U5 0.09 mm to (138.8, 53.3)
Routing:
- net GND: track 174.6 -> 198.2 mm, vias 0 -> 1
- net +5V: track 155.7 -> 160.3 mm
- net +3.3V: track 120.8 -> 125.4 mm
- net LV_D1: track 30.8 -> 35.3 mm
- net D6: track 53.0 -> 55.6 mm
- net LV_GRMCLK: track 17.3 -> 19.8 mm
- net ~{LV_GS}: track 14.9 -> 17.4 mm
- net LV_D2: track 29.5 -> 32.0 mm
- net LV_D3: track 29.5 -> 32.0 mm
- net LV_D0: track 30.9 -> 33.4 mm
- net LV_GREADY: track 38.2 -> 40.7 mm
- net LV_DBIN: track 13.8 -> 16.3 mm
- net LV_A14: track 14.9 -> 17.4 mm
- net D3: track 28.5 -> 30.7 mm
- net D2: track 24.9 -> 27.1 mm
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Other:
- board text added: "Unicorn Board GROM Replacement Dan Werner 11/13/22 V0.9"
- board text removed: "Unicorn Board GROM Replacement Dan Werner 10/14/22 V0.5"

Commit message: hardware updates
Connections:
- U4 pad 11: unconnected-(U4-Pad11) -> ~{LV_RESET}
- U4 pad 2: unconnected-(U4-Pad2) -> ~{RESET}
- U5 pad 7: ~{RESET} -> ~{LV_RESET}
Routing:
- net ~{RESET}: track 35.2 -> 87.6 mm, vias 2 -> 5
- net ~{LV_RESET}: track 0.00 -> 19.8 mm
