File: unicornboard/unicorn/unicorn.kicad_sch (KiCad schematic)
At the start: 6 parts, among them J1 UNICORN PORT, U1 HV-LV, U2 HV-LV, U3 HV-LV, U4 HV-LV, U5 ESP32_MODULE

Commit message: unicorn work
Parts:
- removed J1: UNICORN PORT, Connector_PinHeader_2.54mm:PinHeader_1x15_P2.54mm_Vertical, symbol Connector:Conn_01x15_Male
- added H1, H2, H3, H4: MountingHole, MountingHole:MountingHole_3.2mm_M3, symbol Mechanical:MountingHole
- added J1: UNICORN PORT, Connector_PinHeader_2.54mm:PinHeader_1x16_P2.54mm_Vertical, symbol Connector:Conn_01x16_Male
Connections:
- net +5V: now also J1.14 (Pin_14)
- net D0: now also J1.1 (Pin_1)
- net D1: now also J1.2 (Pin_2)
- net D2: now also J1.3 (Pin_3)
- net D3: now also J1.4 (Pin_4)
- net D4: now also J1.5 (Pin_5)
- net D5: now also J1.6 (Pin_6)
- net D6: now also J1.7 (Pin_7)
- net D7: now also J1.8 (Pin_8)
- net DBIN: now also J1.10 (Pin_10)
- net GND: now also J1.15 (Pin_15)
- net GREADY: now also J1.9 (Pin_9)
- net GRMCLK: now also J1.12 (Pin_12)
- net IO_A14: now also J1.11 (Pin_11)
- net ~{GS}: now also J1.13 (Pin_13)
- net ~{RESET}: now reaches U5.7 (GPIO33)
- net ~{RESET}: now also J1.16 (Pin_16)
- no-connect marks 19 -> 18

Commit message: hardware updates
Connections:
- net ~{RESET}: now also U4.2 (HV3); no longer U5.7 (GPIO33)
- net ~{LV_RESET}: now reaches U4.11 (LV3)
- net ~{LV_RESET}: now also U5.7 (GPIO33)
- no-connect marks 18 -> 16
Changed lines of the file:
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@@
   (title_block
     (title "UNICORN GROM REPLACEMENT")
-    (date "2022-10-14")
-    (rev "V0.5")
+    (date "2022-11-13")
+    (rev "V0.9")
   )
   (junction (at 35.56 64.77) (diameter 0) (color 0 0 0 0)
@@
   (junction (at 22.86 67.31) (diameter 0) (color 0 0 0 0)
   )
-  (no_connect (at 81.28 106.68))
-  (no_connect (at 101.6 106.68))
   (no_connect (at 101.6 114.3))
   (no_connect (at 101.6 116.84))
@@
     (stroke (width 0) (type default) (color 0 0 0 0))
   )
+  (wire (pts (xy 78.74 106.68) (xy 81.28 106.68))
+    (stroke (width 0) (type default) (color 0 0 0 0))
+  )
   (wire (pts (xy 101.6 92.71) (xy 106.68 92.71))
     (stroke (width 0) (type default) (color 0 0 0 0))
   )
   (wire (pts (xy 152.4 57.15) (xy 153.67 57.15))
+    (stroke (width 0) (type default) (color 0 0 0 0))
+  )
+  (wire (pts (xy 101.6 106.68) (xy 106.68 106.68))
     (stroke (width 0) (type default) (color 0 0 0 0))
   )
@@
     )
   )
+  (global_label "~{LV_RESET}" (shape input) (at 106.68 106.68 0) (fields_autoplaced)
+    (effects (font (size 1.27 1.27)) (justify left))
+    (property "Intersheet References" "${INTERSHEET_REFS}" (id 0) (at 117.8591 106.7594 0)
+      (effects (font (size 1.27 1.27)) (justify left) hide)
+    )
+  )
   (global_label "LV_D0" (shape input) (at 182.88 44.45 0) (fields_autoplaced)
     (effects (font (size 1.25 1.25)) (justify left))
@@
     )
   )
-  (global_label "~{RESET}" (shape input) (at 149.86 46.99 180) (fields_autoplaced)
+  (global_label "~{LV_RESET}" (shape input) (at 149.86 46.99 180) (fields_autoplaced)
     (effects (font (size 1.27 1.27)) (justify right))
-    (property "Intersheet References" "${INTERSHEET_REFS}" (id 0) (at 141.7652 46.9106 0)
+    (property "Intersheet References" "${INTERSHEET_REFS}" (id 0) (at 138.6809 46.9106 0)
       (effects (font (size 1.27 1.27)) (justify right) hide)
     )
@@
     )
   )
+  (global_label "~{RESET}" (shape input) (at 78.74 106.68 180) (fields_autoplaced)
+    (effects (font (size 1.27 1.27)) (justify right))
+    (property "Intersheet References" "${INTERSHEET_REFS}" (id 0) (at 70.6452 106.6006 0)
+      (effects (font (size 1.27 1.27)) (justify right) hide)
+    )
+  )
