File: mainboard/Console.kicad_pcb (KiCad board)
At the start: 2 copper layers, 359.4 x 194.3 mm, 305 parts, among them J1 Reset, J10 Joystick, J11 Keyboard, J12 I/O Port, J13 I/O Port, J14 GROM Port, J15 GROM Port, J16 Rom Select 1, J17 Rom Select 2, J2 Power LED, J3 POWER, J4 UNICORN PORT, J5 ROM Select, J6 ROM Select, J7 AUDIO OUT, J8 VIDEO OUT, J9 Cassette, Q1 TIS92, Q2 2N3904, Q3 TIS92, Q4 TIS92, Q5 TIS92, Q6 TIS92, Q7 TIS92, Q8 TIS92, Q9 TIS92, SW1 RAM Size, SW2 Internal Cart ROM Enable, U1 TIM9904, U10 74LS00, U11 74LS244, U12 74LS373, U13 74LS245, U14 74LS00, U15 74LS04, U16 74LS74, U17 74LS194, U18 74LS00, U19 LM7905_TO220, U2 TMS9900, U20 74LS04, U21 74LS04, U22 TMC0430, U23 TMC0430, U24 TMC0430, U25 HM62256BLP, U26 HM62256BLP, U27 27C64, U28 27C64, U29 SN76489, U3 74LS04, U30 TMS9918, U31 74LS574, U32 74LS574, U33 HM62256BLP, U34 74LS574, U35 TMS9901, U36 RC4558, U37 74LS156, U38 TIL119, U39 TIL119, U4 74LS32, U40 74LS244, U41 74LS367, U42 74LS367, U43 74LS379, U44 27C010, U5 74LS138, U6 74LS03, U7 74LS08, U8 74LS138, U9 74LS32, Y1 48.000 MHz, Y2 10.7MHz

Commit message: hardware updates
Parts:
- removed L7: 6.8µH, Resistor_THT:R_Axial_DIN0207_L6.3mm_D2.5mm_P7.62mm_Horizontal
- removed R18: 1kΩ, Resistor_THT:R_Axial_DIN0207_L6.3mm_D2.5mm_P7.62mm_Horizontal
- J13: footprint Library:CardEdge_44Pin_2.54mm_Vertical -> WernerCustomLibrary:44 Pin Card Edge
- SW1: footprint Package_DIP:DIP-10_W10.16mm_LongPads -> Package_DIP:DIP-10_W7.62mm_Socket_LongPads
- moved J13 74.9 mm to (384.4, 44.3), turned to 180 degrees
- moved C60 21.3 mm to (309.1, 58.4)
- moved J8 5.50 mm to (285.0, 34.6)
- moved C52 5.16 mm to (36.9, 53.4)
Connections:
- J3 pad 2: /Power/+5VIN -> +5V
- U5 pad 15: Net-(R18-Pad2) -> ~{ROM}
Other:
- outline, holes or cut-outs redrawn
- board text added: "TI99/22 V0.90 Dan Werner 11/13/22 http://github.com/danwerner21/ti99_22"
- board text removed: "TI99/22 V0.90 Dan Werner 11/5/22 http://github.com/danwerner21/ti99_22"

Commit message: hardware updates
Parts:
- U44: value 27C010 -> 27C010-C
- moved U44 3.58 mm to (63.6, 176.8)
- renumbered L11 to L10, L12 to L11, L13 to L12, L14 to L13, L15 to L14, L16 to L15, L17 to L16, L18 to L17, L19 to L18, L20 to L19, L21 to L20, L22 to L21, L8 to L7, L9 to L8, L10 to L9, R101 to R100, R19 to R18, R20 to R19, R21 to R20, R22 to R21, R23 to R22, R24 to R23, R25 to R24, R26 to R25, R27 to R26, R28 to R27, R29 to R28, R30 to R29, R31 to R30, R32 to R31, R33 to R32, R34 to R33, R35 to R34, R36 to R35, R37 to R36, R38 to R37, R39 to R38, R40 to R39, R41 to R40, R42 to R41, R43 to R42, R44 to R43, R45 to R44, R46 to R45, R47 to R46, R48 to R47, R49 to R48, R50 to R49, R51 to R50, R52 to R51, R53 to R52, R54 to R53, R55 to R54, R56 to R55, R57 to R56, R58 to R57, R59 to R58, R60 to R59, R61 to R60, R62 to R61, R63 to R62, R64 to R63, R65 to R64, R66 to R65, R67 to R66, R68 to R67, R69 to R68, R70 to R69, R71 to R70, R72 to R71, R73 to R72, R74 to R73, R75 to R74, R76 to R75, R77 to R76, R78 to R77, R79 to R78, R80 to R79, R81 to R80, R82 to R81, R83 to R82, R84 to R83, R85 to R84, R86 to R85, R87 to R86, R88 to R87, R89 to R88, R90 to R89, R91 to R90, R92 to R91, R93 to R92, R94 to R93, R95 to R94, R96 to R95, R97 to R96, R98 to R97, R99 to R98, R100 to R99
Connections:
- U44 pad 30: (no net) -> +5V
Other:
- board text added: "+12"
- board text added: "+5"
- board text added: "-12"
- board text added: "GND"

Commit message: Add BOM
Parts:
- J10, J9: footprint Connector_Dsub:DSUB-9_Male_Horizontal_P2.77x2.84mm_EdgePinOffset14.56mm_Housed_MountingHolesOffset8.20mm -> Connector_Dsub:DSUB-9_Female_Horizontal_P2.77x2.84mm_EdgePinOffset4.94mm_Housed_MountingHolesOffset7.48mm
- moved C16 155.6 mm to (171.5, 179.5)
- moved R94 66.1 mm to (293.4, 34.4)
- moved C59 61.4 mm to (297.5, 124.6)
- moved C60 44.7 mm to (269.6, 79.5)
- moved C61 35.0 mm to (296.0, 95.5)
- moved R29 30.7 mm to (322.0, 109.5), turned to 90 degrees
- moved C24 26.7 mm to (332.0, 95.0)
- moved J10 24.4 mm to (32.6, 158.2)
- moved L10 24.1 mm to (301.5, 87.5), turned to 180 degrees
- moved R33 15.2 mm to (287.8, 79.1), turned to 180 degrees
- moved R31 14.8 mm to (301.6, 76.4)
- moved Q2 14.3 mm to (292.8, 78.9)
- moved U42 12.3 mm to (330.6, 70.6)
- moved R30 10.1 mm to (306.3, 85.4)
- moved J9 8.10 mm to (32.5, 95.5)
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Other:
- board size 359.4 x 194.3 mm -> 350 x 194.3 mm
- board text added: "GROM Chips optional with attached UNICORN board"
- board text added: "Only populate one, header for remote cart slot or on-board slot"
