File: mainboard/Keyboard.kicad_sch (KiCad schematic)
At the start: 20 parts, among them J10 Joystick, J11 Keyboard, U19 LM2901, U21 LM2903, U39 TMS9901, U40 74LS156

Commit message: PCB 0.96
Parts:
- J10: footprint Connector_Dsub:DSUB-9_Female_Horizontal_P2.77x2.84mm_EdgePinOffset4.94mm_Housed_MountingHolesOffset7.48mm -> Connector_Dsub:DSUB-9_Male_Horizontal_P2.77x2.84mm_EdgePinOffset4.94mm_Housed_MountingHolesOffset7.48mm
- R36, R37, R38, R39, R40: value 100kΩ -> 100Ω
Changed lines of the file:
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@@
   (title_block
     (title "TI-99/22")
-    (date "2022-12-26")
-    (rev "0.95")
+    (date "2023-01-21")
+    (rev "0.96")
     (company "Dan Werner - https://github.com/danwerner21/ti99_22")
     (comment 1 "Schematic for Keyboard, Joystick and Cassette port.")
@@
       (effects (font (size 1.778 1.778)))
     )
-    (property "Footprint" "Connector_Dsub:DSUB-9_Female_Horizontal_P2.77x2.84mm_EdgePinOffset4.94mm_Housed_MountingHolesOffset7.48mm" (id 2) (at 141.224 34.036 0)
+    (property "Footprint" "Connector_Dsub:DSUB-9_Male_Horizontal_P2.77x2.84mm_EdgePinOffset4.94mm_Housed_MountingHolesOffset7.48mm" (id 2) (at 141.224 34.036 0)
       (effects (font (size 1.524 1.524)) hide)
     )
@@
     (in_bom yes) (on_board yes)
     (property "Reference" "R40" (id 0) (at 191.262 126.746 90))
-    (property "Value" "100kΩ" (id 1) (at 192.532 124.46 90))
+    (property "Value" "100Ω" (id 1) (at 192.532 124.46 90))
     (property "Footprint" "Resistor_THT:R_Axial_DIN0207_L6.3mm_D2.5mm_P7.62mm_Horizontal" (id 2) (at 192.278 128.524 90)
       (effects (font (size 1.27 1.27)) hide)
@@
     (in_bom yes) (on_board yes)
     (property "Reference" "R39" (id 0) (at 191.262 122.428 90))
-    (property "Value" "100kΩ" (id 1) (at 192.532 120.396 90))
+    (property "Value" "100Ω" (id 1) (at 192.532 120.396 90))
     (property "Footprint" "Resistor_THT:R_Axial_DIN0207_L6.3mm_D2.5mm_P7.62mm_Horizontal" (id 2) (at 192.278 124.206 90)
       (effects (font (size 1.27 1.27)) hide)
@@
     (in_bom yes) (on_board yes)
     (property "Reference" "R37" (id 0) (at 191.008 114.046 90))
-    (property "Value" "100kΩ" (id 1) (at 192.278 112.014 90))
+    (property "Value" "100Ω" (id 1) (at 192.278 112.014 90))
     (property "Footprint" "Resistor_THT:R_Axial_DIN0207_L6.3mm_D2.5mm_P7.62mm_Horizontal" (id 2) (at 192.278 115.824 90)
       (effects (font (size 1.27 1.27)) hide)
@@
     (in_bom yes) (on_board yes)
     (property "Reference" "R36" (id 0) (at 191.008 109.982 90))
-    (property "Value" "100kΩ" (id 1) (at 192.278 107.95 90))
+    (property "Value" "100Ω" (id 1) (at 192.278 107.95 90))
     (property "Footprint" "Resistor_THT:R_Axial_DIN0207_L6.3mm_D2.5mm_P7.62mm_Horizontal" (id 2) (at 192.278 111.76 90)
       (effects (font (size 1.27 1.27)) hide)
@@
     (in_bom yes) (on_board yes)
     (property "Reference" "R38" (id 0) (at 191.008 118.364 90))
-    (property "Value" "100kΩ" (id 1) (at 192.532 116.332 90))
+    (property "Value" "100Ω" (id 1) (at 192.532 116.332 90))
     (property "Footprint" "Resistor_THT:R_Axial_DIN0207_L6.3mm_D2.5mm_P7.62mm_Horizontal" (id 2) (at 192.278 120.142 90)
       (effects (font (size 1.27 1.27)) hide)
