File: mainboard/8bit16bitSwitch.kicad_sch (KiCad schematic)
At the start: 13 parts, among them U10 74LS00, U11 74LS244, U12 74LS373, U13 74LS245, U14 74LS00, U15 74LS04, U16 74LS74, U17 74LS194, U18 74LS00, U3 74LS04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

Commit message: PCB routed
Parts:
- U10, U14, U15, U16, U18, U3, U4: footprint Package_DIP:DIP-14_W7.62mm_LongPads -> Package_DIP:DIP-14_W7.62mm_Socket_LongPads
- U11, U12, U13: footprint Package_DIP:DIP-20_W7.62mm_LongPads -> Package_DIP:DIP-20_W7.62mm_Socket_LongPads
- U17: footprint Package_DIP:DIP-16_W7.62mm_LongPads -> Package_DIP:DIP-16_W7.62mm_Socket_LongPads
Changed lines of the file:
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@@
       (effects (font (size 1.524 1.524)) (justify left top))
     )
-    (property "Footprint" "Package_DIP:DIP-20_W7.62mm_LongPads" (id 2) (at 96.52 116.84 0)
+    (property "Footprint" "Package_DIP:DIP-20_W7.62mm_Socket_LongPads" (id 2) (at 96.52 116.84 0)
       (effects (font (size 1.524 1.524)) hide)
     )
@@
       (effects (font (size 1.524 1.524)))
     )
-    (property "Footprint" "Package_DIP:DIP-20_W7.62mm_LongPads" (id 2) (at 95.25 67.31 0)
+    (property "Footprint" "Package_DIP:DIP-20_W7.62mm_Socket_LongPads" (id 2) (at 95.25 67.31 0)
       (effects (font (size 1.524 1.524)) hide)
     )
@@
       (effects (font (size 1.524 1.524)))
     )
-    (property "Footprint" "Package_DIP:DIP-20_W7.62mm_LongPads" (id 2) (at 60.96 167.64 0)
+    (property "Footprint" "Package_DIP:DIP-20_W7.62mm_Socket_LongPads" (id 2) (at 60.96 167.64 0)
       (effects (font (size 1.524 1.524)) hide)
     )
@@
       (effects (font (size 1.524 1.524)))
     )
-    (property "Footprint" "Package_DIP:DIP-14_W7.62mm_LongPads" (id 2) (at 170.18 60.96 0)
+    (property "Footprint" "Package_DIP:DIP-14_W7.62mm_Socket_LongPads" (id 2) (at 170.18 60.96 0)
       (effects (font (size 1.524 1.524)) hide)
     )
@@
       (effects (font (size 1.524 1.524)))
     )
-    (property "Footprint" "Package_DIP:DIP-14_W7.62mm_LongPads" (id 2) (at 161.29 83.82 0)
+    (property "Footprint" "Package_DIP:DIP-14_W7.62mm_Socket_LongPads" (id 2) (at 161.29 83.82 0)
       (effects (font (size 1.524 1.524)) hide)
     )
@@
       (effects (font (size 1.524 1.524)))
     )
-    (property "Footprint" "Package_DIP:DIP-14_W7.62mm_LongPads" (id 2) (at 241.3 85.09 0)
+    (property "Footprint" "Package_DIP:DIP-14_W7.62mm_Socket_LongPads" (id 2) (at 241.3 85.09 0)
       (effects (font (size 1.524 1.524)) hide)
     )
@@
       (effects (font (size 1.524 1.524)))
     )
-    (property "Footprint" "Package_DIP:DIP-16_W7.62mm_LongPads" (id 2) (at 204.47 87.63 0)
+    (property "Footprint" "Package_DIP:DIP-16_W7.62mm_Socket_LongPads" (id 2) (at 204.47 87.63 0)
       (effects (font (size 1.524 1.524)) hide)
     )
@@
       (effects (font (size 1.524 1.524)))
     )
-    (property "Footprint" "Package_DIP:DIP-14_W7.62mm_LongPads" (id 2) (at 38.1 180.34 0)
+    (property "Footprint" "Package_DIP:DIP-14_W7.62mm_Socket_LongPads" (id 2) (at 38.1 180.34 0)
       (effects (font (size 1.524 1.524)) hide)
     )
@@
       (effects (font (size 1.524 1.524)))
     )
-    (property "Footprint" "Package_DIP:DIP-14_W7.62mm_LongPads" (id 2) (at 140.97 118.11 0)
+    (property "Footprint" "Package_DIP:DIP-14_W7.62mm_Socket_LongPads" (id 2) (at 140.97 118.11 0)
       (effects (font (size 1.524 1.524)) hide)
     )
@@
       (effects (font (size 1.524 1.524)))
     )
-    (property "Footprint" "Package_DIP:DIP-14_W7.62mm_LongPads" (id 2) (at 140.97 129.54 0)
+    (property "Footprint" "Package_DIP:DIP-14_W7.62mm_Socket_LongPads" (id 2) (at 140.97 129.54 0)
       (effects (font (size 1.524 1.524)) hide)
     )
@@
       (effects (font (size 1.524 1.524)))
     )
-    (property "Footprint" "Package_DIP:DIP-14_W7.62mm_LongPads" (id 2) (at 224.79 128.27 0)
+    (property "Footprint" "Package_DIP:DIP-14_W7.62mm_Socket_LongPads" (id 2) (at 224.79 128.27 0)
       (effects (font (size 1.524 1.524)) hide)
     )
@@
       (effects (font (size 1.524 1.524)))
     )
-    (property "Footprint" "Package_DIP:DIP-14_W7.62mm_LongPads" (id 2) (at 240.03 128.27 0)
+    (property "Footprint" "Package_DIP:DIP-14_W7.62mm_Socket_LongPads" (id 2) (at 240.03 128.27 0)
       (effects (font (size 1.524 1.524)) hide)
     )
@@
       (effects (font (size 1.524 1.524)))
     )
-    (property "Footprint" "Package_DIP:DIP-14_W7.62mm_LongPads" (id 2) (at 113.03 160.02 0)
+    (property "Footprint" "Package_DIP:DIP-14_W7.62mm_Socket_LongPads" (id 2) (at 113.03 160.02 0)
       (effects (font (size 1.524 1.524)) hide)
     )
@@
       (effects (font (size 1.524 1.524)))
     )
-    (property "Footprint" "Package_DIP:DIP-14_W7.62mm_LongPads" (id 2) (at 204.47 137.16 0)
+    (property "Footprint" "Package_DIP:DIP-14_W7.62mm_Socket_LongPads" (id 2) (at 204.47 137.16 0)
       (effects (font (size 1.524 1.524)) hide)
     )
@@
       (effects (font (size 1.524 1.524)))
     )
-    (property "Footprint" "Package_DIP:DIP-14_W7.62mm_LongPads" (id 2) (at 160.02 162.56 0)
+    (property "Footprint" "Package_DIP:DIP-14_W7.62mm_Socket_LongPads" (id 2) (at 160.02 162.56 0)
       (effects (font (size 1.524 1.524)) hide)
     )
@@
       (effects (font (size 1.524 1.524)))
     )
-    (property "Footprint" "Package_DIP:DIP-14_W7.62mm_LongPads" (id 2) (at 135.89 162.56 0)
+    (property "Footprint" "Package_DIP:DIP-14_W7.62mm_Socket_LongPads" (id 2) (at 135.89 162.56 0)
       (effects (font (size 1.524 1.524)) hide)
     )
@@
       (effects (font (size 1.524 1.524)))
     )
-    (property "Footprint" "Package_DIP:DIP-14_W7.62mm_LongPads" (id 2) (at 245.11 101.6 0)
+    (property "Footprint" "Package_DIP:DIP-14_W7.62mm_Socket_LongPads" (id 2) (at 245.11 101.6 0)
       (effects (font (size 1.524 1.524)) hide)
     )
@@
       (effects (font (size 1.524 1.524)))
     )
-    (property "Footprint" "Package_DIP:DIP-14_W7.62mm_LongPads" (id 2) (at 245.11 114.3 0)
+    (property "Footprint" "Package_DIP:DIP-14_W7.62mm_Socket_LongPads" (id 2) (at 245.11 114.3 0)
       (effects (font (size 1.524 1.524)) hide)
     )
@@
       (effects (font (size 1.524 1.524)))
     )
-    (property "Footprint" "Package_DIP:DIP-14_W7.62mm_LongPads" (id 2) (at 243.84 38.1 0)
+    (property "Footprint" "Package_DIP:DIP-14_W7.62mm_Socket_LongPads" (id 2) (at 243.84 38.1 0)
       (effects (font (size 1.524 1.524)) hide)
     )
@@
       (effects (font (size 1.524 1.524)))
     )
-    (property "Footprint" "Package_DIP:DIP-14_W7.62mm_LongPads" (id 2) (at 259.08 40.64 0)
+    (property "Footprint" "Package_DIP:DIP-14_W7.62mm_Socket_LongPads" (id 2) (at 259.08 40.64 0)
       (effects (font (size 1.524 1.524)) hide)
     )
@@
       (effects (font (size 1.524 1.524)))
     )
-    (property "Footprint" "Package_DIP:DIP-14_W7.62mm_LongPads" (id 2) (at 245.11 62.23 0)
-      (effects (font (size 1.524 1.524)) hide)
-    )
+    (property "Footprint" "Package_DIP:DIP-14_W7.62mm_Socket_LongPads" (id 2) (at 245.11 62.23 0)
+      (effects (font (size 1.524 1.524)) hide)
+    )

Commit message: unicorn work
Changed lines of the file:
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@@
   (title_block
     (title "TI-99/22")
-    (date "2022-06-23")
-    (rev "0.75")
+    (date "2022-10-11")
+    (rev "0.76")
     (company "Dan Werner - https://github.com/danwerner21/ti99_22")
     (comment 1 "Logic for generating the Address line 15 and multiplexing the Databus")
@@
       (effects (font (size 1.524 1.524)))
     )
-    (pin "10")
-    (pin "11")
+    (pin "1")
+    (pin "2")
+    (pin "3")
+    (pin "4")
+    (pin "5")
+    (pin "6")
+    (pin "8")
+    (pin "9")
+    (pin "10")
+    (pin "11")
+    (pin "12")
+    (pin "13")
+    (pin "14")
+    (pin "7")
   )
   (symbol (lib_id "74xx:74LS74") (at 161.29 83.82 0) (mirror x) (unit 2)
@@
       (effects (font (size 1.524 1.524)))
     )
-    (pin "10")
-    (pin "11")
-    (pin "12")
-    (pin "13")
-    (pin "8")
-    (pin "9")
+    (pin "1")
+    (pin "2")
+    (pin "3")
+    (pin "4")
+    (pin "5")
+    (pin "6")
+    (pin "10")
+    (pin "11")
+    (pin "12")
+    (pin "13")
+    (pin "8")
+    (pin "9")
+    (pin "14")
+    (pin "7")
   )
   (symbol (lib_id "Console-rescue:+5V") (at 161.29 76.2 0) (unit 1)
@@
       (effects (font (size 1.524 1.524)))
     )
-    (pin "8")
-    (pin "9")
+    (pin "1")
+    (pin "2")
+    (pin "3")
+    (pin "4")
+    (pin "5")
+    (pin "6")
+    (pin "8")
+    (pin "9")
+    (pin "10")
+    (pin "11")
+    (pin "12")
+    (pin "13")
+    (pin "14")
+    (pin "7")
   )
   (symbol (lib_id "74xx:74LS194") (at 204.47 87.63 0) (unit 1)
@@
       (effects (font (size 1.524 1.524)))
     )
-    (pin "10")
-    (pin "8")
-    (pin "9")
+    (pin "1")
+    (pin "2")
+    (pin "3")
+    (pin "4")
+    (pin "5")
+    (pin "6")
+    (pin "10")
+    (pin "8")
+    (pin "9")
+    (pin "11")
+    (pin "12")
+    (pin "13")
+    (pin "14")
+    (pin "7")
   )
   (symbol (lib_id "74xx:74LS00") (at 140.97 118.11 0) (mirror y) (unit 2)
@@
       (effects (font (size 1.524 1.524)))
     )
-    (property "Value" "74LS00" (id 1) (at 140.97 120.65 0)
+    (property "Value" "74LS00" (id 1) (at 140.97 113.03 0)
       (effects (font (size 1.524 1.524)))
     )
@@
       (effects (font (size 1.524 1.524)))
     )
-    (pin "4")
-    (pin "5")
-    (pin "6")
+    (pin "1")
+    (pin "2")
+    (pin "3")
+    (pin "4")
+    (pin "5")
+    (pin "6")
+    (pin "10")
+    (pin "8")
+    (pin "9")
+    (pin "11")
+    (pin "12")
+    (pin "13")
+    (pin "14")
+    (pin "7")
   )
   (symbol (lib_id "74xx:74LS00") (at 140.97 129.54 0) (mirror y) (unit 2)
@@
       (effects (font (size 1.524 1.524)))
     )
-    (property "Value" "74LS00" (id 1) (at 140.97 132.08 0)
+    (property "Value" "74LS00" (id 1) (at 140.97 124.46 0)
       (effects (font (size 1.524 1.524)))
     )
@@
       (effects (font (size 1.524 1.524)))
     )
-    (pin "4")
-    (pin "5")
-    (pin "6")
+    (pin "1")
+    (pin "2")
+    (pin "3")
+    (pin "4")
+    (pin "5")
+    (pin "6")
+    (pin "10")
+    (pin "8")
+    (pin "9")
+    (pin "11")
+    (pin "12")
+    (pin "13")
+    (pin "14")
+    (pin "7")
   )
   (symbol (lib_id "74xx:74LS00") (at 224.79 128.27 0) (mirror x) (unit 4)
@@
       (effects (font (size 1.524 1.524)))
     )
-    (property "Value" "74LS00" (id 1) (at 224.79 125.73 0)
+    (property "Value" "74LS00" (id 1) (at 224.79 123.19 0)
       (effects (font (size 1.524 1.524)))
     )
@@
       (effects (font (size 1.524 1.524)))
     )
-    (pin "11")
-    (pin "12")
-    (pin "13")
+    (pin "1")
+    (pin "2")
+    (pin "3")
+    (pin "4")
+    (pin "5")
+    (pin "6")
+    (pin "10")
+    (pin "8")
+    (pin "9")
+    (pin "11")
+    (pin "12")
+    (pin "13")
+    (pin "14")
+    (pin "7")
   )
   (symbol (lib_id "74xx:74LS04") (at 240.03 128.27 0) (unit 2)
@@
       (effects (font (size 1.524 1.524)))
     )
-    (pin "3")
-    (pin "4")
+    (pin "1")
+    (pin "2")
+    (pin "3")
+    (pin "4")
+    (pin "5")
+    (pin "6")
+    (pin "8")
+    (pin "9")
+    (pin "10")
+    (pin "11")
+    (pin "12")
+    (pin "13")
+    (pin "14")
+    (pin "7")
   )
   (symbol (lib_id "74xx:74LS00") (at 113.03 160.02 0) (unit 4)
@@
       (effects (font (size 1.524 1.524)))
     )
-    (pin "11")
-    (pin "12")
-    (pin "13")
+    (pin "1")
+    (pin "2")
+    (pin "3")
+    (pin "4")
+    (pin "5")
+    (pin "6")
+    (pin "10")
+    (pin "8")
+    (pin "9")
+    (pin "11")
+    (pin "12")
+    (pin "13")
+    (pin "14")
+    (pin "7")
   )
   (symbol (lib_id "74xx:74LS00") (at 204.47 137.16 0) (mirror x) (unit 1)
@@
       (effects (font (size 1.524 1.524)))
     )
-    (property "Value" "74LS00" (id 1) (at 204.47 134.62 0)
+    (property "Value" "74LS00" (id 1) (at 204.47 132.08 0)
       (effects (font (size 1.524 1.524)))
     )
@@
     (pin "2")
     (pin "3")
+    (pin "4")
+    (pin "5")
+    (pin "6")
+    (pin "10")
+    (pin "8")
+    (pin "9")
+    (pin "11")
+    (pin "12")
+    (pin "13")
+    (pin "14")
+    (pin "7")
   )
   (symbol (lib_id "74xx:74LS04") (at 160.02 162.56 0) (unit 1)
@@
     (pin "1")
     (pin "2")
+    (pin "3")
+    (pin "4")
+    (pin "5")
+    (pin "6")
+    (pin "8")
+    (pin "9")
+    (pin "10")
+    (pin "11")
+    (pin "12")
+    (pin "13")
+    (pin "14")
+    (pin "7")
   )
   (symbol (lib_id "74xx:74LS32") (at 135.89 162.56 0) (mirror x) (unit 4)
@@
       (effects (font (size 1.524 1.524)))
     )
-    (pin "11")
-    (pin "12")
-    (pin "13")
+    (pin "1")
+    (pin "2")
+    (pin "3")
+    (pin "4")
+    (pin "5")
+    (pin "6")
+    (pin "10")
+    (pin "8")
+    (pin "9")
+    (pin "11")
+    (pin "12")
+    (pin "13")
+    (pin "14")
+    (pin "7")
   )
   (symbol (lib_id "74xx:74LS00") (at 245.11 101.6 0) (unit 1)
@@
       (effects (font (size 1.524 1.524)))
     )
-    (property "Value" "74LS00" (id 1) (at 245.11 104.14 0)
+    (property "Value" "74LS00" (id 1) (at 245.11 96.52 0)
       (effects (font (size 1.524 1.524)))
     )
@@
     (pin "2")
     (pin "3")
+    (pin "4")
+    (pin "5")
+    (pin "6")
+    (pin "10")
+    (pin "8")
+    (pin "9")
+    (pin "11")
+    (pin "12")
+    (pin "13")
+    (pin "14")
+    (pin "7")
   )
   (symbol (lib_id "Console-rescue:+5V") (at 237.49 99.06 90) (unit 1)
@@
       (effects (font (size 1.524 1.524)))
     )
-    (property "Value" "74LS00" (id 1) (at 245.11 116.84 0)
+    (property "Value" "74LS00" (id 1) (at 245.11 119.38 0)
       (effects (font (size 1.524 1.524)))
     )
@@
       (effects (font (size 1.524 1.524)))
     )
-    (pin "4")
-    (pin "5")
-    (pin "6")
+    (pin "1")
+    (pin "2")
+    (pin "3")
+    (pin "4")
+    (pin "5")
+    (pin "6")
+    (pin "10")
+    (pin "8")
+    (pin "9")
+    (pin "11")
+    (pin "12")
+    (pin "13")
+    (pin "14")
+    (pin "7")
   )
   (symbol (lib_id "74xx:74LS04") (at 243.84 38.1 0) (unit 3)
@@
       (effects (font (size 1.524 1.524)))
     )
-    (pin "5")
-    (pin "6")
+    (pin "1")
+    (pin "2")
+    (pin "3")
+    (pin "4")
+    (pin "5")
+    (pin "6")
+    (pin "8")
+    (pin "9")
+    (pin "10")
+    (pin "11")
+    (pin "12")
+    (pin "13")
+    (pin "14")
+    (pin "7")
   )
   (symbol (lib_id "74xx:74LS00") (at 259.08 40.64 0) (mirror x) (unit 1)
@@
     (pin "2")
     (pin "3")
+    (pin "4")
+    (pin "5")
+    (pin "6")
+    (pin "10")
+    (pin "8")
+    (pin "9")
+    (pin "11")
+    (pin "12")
+    (pin "13")
+    (pin "14")
+    (pin "7")
   )
   (symbol (lib_id "74xx:74LS74") (at 245.11 62.23 0) (unit 1)
@@
     (pin "5")
     (pin "6")
+    (pin "10")
+    (pin "11")
+    (pin "12")
+    (pin "13")
+    (pin "8")
+    (pin "9")
+    (pin "14")
+    (pin "7")
   )
   (symbol (lib_id "Console-rescue:GND") (at 204.47 113.03 0) (unit 1)

Commit message: PCB cleanup
Parts:
- C13, C14: symbol TI-Customs:C_Small -> Device:C
Other:
- moved on the sheet: C13, C14
