File: mainboard/AddressDecoding.kicad_sch (KiCad schematic)
At the start: 16 parts, among them SW1 RAM Size, U5 74LS138, U6 74LS03, U7 74LS32, U8 74LS138, U9 74LS32

Commit message: PCB routed
Parts:
- SW1: footprint (none) -> Package_DIP:DIP-10_W10.16mm_LongPads
- U5, U8: footprint Package_DIP:DIP-16_W7.62mm_LongPads -> Package_DIP:DIP-16_W7.62mm_Socket_LongPads
- U6, U7: footprint Package_DIP:DIP-14_W7.62mm_LongPads -> Package_DIP:DIP-14_W7.62mm_Socket_LongPads
- U9: footprint Package_DIP:DIP-16_W7.62mm_LongPads -> Package_DIP:DIP-14_W7.62mm_Socket_LongPads
Changed lines of the file:
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@@
       (effects (font (size 1.524 1.524)))
     )
-    (property "Footprint" "Package_DIP:DIP-16_W7.62mm_LongPads" (id 2) (at 135.89 67.31 0)
+    (property "Footprint" "Package_DIP:DIP-16_W7.62mm_Socket_LongPads" (id 2) (at 135.89 67.31 0)
       (effects (font (size 1.524 1.524)) hide)
     )
@@
       (effects (font (size 1.524 1.524)))
     )
-    (property "Footprint" "Package_DIP:DIP-14_W7.62mm_LongPads" (id 2) (at 105.41 72.39 0)
+    (property "Footprint" "Package_DIP:DIP-14_W7.62mm_Socket_LongPads" (id 2) (at 105.41 72.39 0)
       (effects (font (size 1.524 1.524)) hide)
     )
@@
       (effects (font (size 1.524 1.524)))
     )
-    (property "Footprint" "Package_DIP:DIP-16_W7.62mm_LongPads" (id 2) (at 99.06 113.03 0)
+    (property "Footprint" "Package_DIP:DIP-16_W7.62mm_Socket_LongPads" (id 2) (at 99.06 113.03 0)
       (effects (font (size 1.524 1.524)) hide)
     )
@@
       (effects (font (size 1.524 1.524)))
     )
-    (property "Footprint" "Package_DIP:DIP-14_W7.62mm_LongPads" (id 2) (at 173.99 72.39 0)
+    (property "Footprint" "Package_DIP:DIP-14_W7.62mm_Socket_LongPads" (id 2) (at 173.99 72.39 0)
       (effects (font (size 1.524 1.524)) hide)
     )
@@
       (effects (font (size 1.524 1.524)))
     )
-    (property "Footprint" "Package_DIP:DIP-14_W7.62mm_LongPads" (id 2) (at 173.99 87.63 0)
+    (property "Footprint" "Package_DIP:DIP-14_W7.62mm_Socket_LongPads" (id 2) (at 173.99 87.63 0)
       (effects (font (size 1.524 1.524)) hide)
     )
@@
       (effects (font (size 1.524 1.524)))
     )
-    (property "Footprint" "Package_DIP:DIP-16_W7.62mm_LongPads" (id 2) (at 212.09 120.65 0)
+    (property "Footprint" "Package_DIP:DIP-14_W7.62mm_Socket_LongPads" (id 2) (at 212.09 120.65 0)
       (effects (font (size 1.524 1.524)) hide)
     )
@@
       (effects (font (size 1.524 1.524)))
     )
-    (property "Footprint" "Package_DIP:DIP-16_W7.62mm_LongPads" (id 2) (at 187.96 123.19 0)
+    (property "Footprint" "Package_DIP:DIP-14_W7.62mm_Socket_LongPads" (id 2) (at 187.96 123.19 0)
       (effects (font (size 1.524 1.524)) hide)
     )
@@
       (effects (font (size 1.524 1.524)))
     )
-    (property "Footprint" "Package_DIP:DIP-16_W7.62mm_LongPads" (id 2) (at 172.72 128.27 0)
+    (property "Footprint" "Package_DIP:DIP-14_W7.62mm_Socket_LongPads" (id 2) (at 172.72 128.27 0)
       (effects (font (size 1.524 1.524)) hide)
     )
@@
     (property "Reference" "U7" (id 0) (at 160.02 144.78 0))
     (property "Value" "74LS32" (id 1) (at 160.02 147.32 0))
-    (property "Footprint" "Package_DIP:DIP-14_W7.62mm_LongPads" (id 2) (at 160.02 153.67 0)
+    (property "Footprint" "Package_DIP:DIP-14_W7.62mm_Socket_LongPads" (id 2) (at 160.02 153.67 0)
       (effects (font (size 1.27 1.27)) hide)
     )
@@
     (property "Reference" "U7" (id 0) (at 143.51 156.21 0))
     (property "Value" "74LS32" (id 1) (at 143.51 158.75 0))
-    (property "Footprint" "Package_DIP:DIP-14_W7.62mm_LongPads" (id 2) (at 143.51 165.1 0)
+    (property "Footprint" "Package_DIP:DIP-14_W7.62mm_Socket_LongPads" (id 2) (at 143.51 165.1 0)
       (effects (font (size 1.27 1.27)) hide)
     )
@@
     (property "Reference" "U7" (id 0) (at 124.46 139.7 0))
     (property "Value" "74LS32" (id 1) (at 124.46 142.24 0))
-    (property "Footprint" "Package_DIP:DIP-14_W7.62mm_LongPads" (id 2) (at 124.46 148.59 0)
+    (property "Footprint" "Package_DIP:DIP-14_W7.62mm_Socket_LongPads" (id 2) (at 124.46 148.59 0)
       (effects (font (size 1.27 1.27)) hide)
     )
@@
     (property "Reference" "SW1" (id 0) (at 80.01 143.51 0))
     (property "Value" "RAM Size" (id 1) (at 80.01 146.05 0))
-    (property "Footprint" "" (id 2) (at 80.01 156.21 0)
+    (property "Footprint" "Package_DIP:DIP-10_W10.16mm_LongPads" (id 2) (at 80.01 156.21 0)
       (effects (font (size 1.27 1.27)) hide)
     )
@@
     (property "Reference" "U7" (id 0) (at 124.46 165.1 0))
     (property "Value" "74LS32" (id 1) (at 124.46 162.56 0))
-    (property "Footprint" "Package_DIP:DIP-14_W7.62mm_LongPads" (id 2) (at 124.46 157.48 0)
-      (effects (font (size 1.27 1.27)) hide)
-    )
+    (property "Footprint" "Package_DIP:DIP-14_W7.62mm_Socket_LongPads" (id 2) (at 124.46 157.48 0)
+      (effects (font (size 1.27 1.27)) hide)
+    )

Commit message: unicorn work
Parts:
- removed U7: 74LS32, Package_DIP:DIP-14_W7.62mm_Socket_LongPads, symbol 74xx:74LS32
- added U7: 74LS08, Package_DIP:DIP-14_W7.62mm_Socket_LongPads, symbol 74xx:74LS08
Connections:
- net ~{RAM}: now also U7.3
- net at R14.1, SW1.8: now also U7.9
- net at R16.1, SW1.6: now also U7.13
- net at R12.1, SW1.10: now also U7.4
- net at R13.1, SW1.9: now also U7.5
- net at R15.1, SW1.7: now also U7.10
- new net: U7.12, U7.8
- new net: U7.1, U7.6
- new net: U7.11, U7.2
Changed lines of the file:
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@@
   (title_block
     (title "TI-99/22")
-    (date "2022-06-23")
-    (rev "0.75")
+    (date "2022-10-11")
+    (rev "0.76")
     (company "Dan Werner - https://github.com/danwerner21/ti99_22")
     (comment 1 "Address Decoding")
@@
       (effects (font (size 1.524 1.524)))
     )
-    (pin "4")
-    (pin "5")
-    (pin "6")
+    (pin "1")
+    (pin "2")
+    (pin "3")
+    (pin "4")
+    (pin "5")
+    (pin "6")
+    (pin "10")
+    (pin "8")
+    (pin "9")
+    (pin "11")
+    (pin "12")
+    (pin "13")
+    (pin "14")
+    (pin "7")
   )
   (symbol (lib_id "74xx:74LS138") (at 99.06 113.03 0) (unit 1)
@@
       (effects (font (size 1.524 1.524)))
     )
-    (pin "10")
-    (pin "8")
-    (pin "9")
-  )
-  (symbol (lib_id "74xx:74LS03") (at 173.99 87.63 0) (unit 4)
-    (in_bom yes) (on_board yes)
-    (property "Reference" "U6" (id 0) (at 173.99 86.36 0)
-      (effects (font (size 1.524 1.524)))
-    )
-    (property "Value" "74LS03" (id 1) (at 173.99 88.9 0)
-      (effects (font (size 1.524 1.524)))
-    )
-    (property "Footprint" "Package_DIP:DIP-14_W7.62mm_Socket_LongPads" (id 2) (at 173.99 87.63 0)
-      (effects (font (size 1.524 1.524)) hide)
-    )
-    (property "Datasheet" "" (id 3) (at 173.99 87.63 0)
-      (effects (font (size 1.524 1.524)))
-    )
+    (pin "1")
+    (pin "2")
+    (pin "3")
+    (pin "4")
+    (pin "5")
+    (pin "6")
+    (pin "10")
+    (pin "8")
+    (pin "9")
     (pin "11")
     (pin "12")
     (pin "13")
+    (pin "14")
+    (pin "7")
+  )
+  (symbol (lib_id "74xx:74LS03") (at 173.99 87.63 0) (unit 4)
+    (in_bom yes) (on_board yes)
+    (property "Reference" "U6" (id 0) (at 173.99 86.36 0)
+      (effects (font (size 1.524 1.524)))
+    )
+    (property "Value" "74LS03" (id 1) (at 173.99 88.9 0)
+      (effects (font (size 1.524 1.524)))
+    )
+    (property "Footprint" "Package_DIP:DIP-14_W7.62mm_Socket_LongPads" (id 2) (at 173.99 87.63 0)
+      (effects (font (size 1.524 1.524)) hide)
+    )
+    (property "Datasheet" "" (id 3) (at 173.99 87.63 0)
+      (effects (font (size 1.524 1.524)))
+    )
+    (pin "1")
+    (pin "2")
+    (pin "3")
+    (pin "4")
+    (pin "5")
+    (pin "6")
+    (pin "10")
+    (pin "8")
+    (pin "9")
+    (pin "11")
+    (pin "12")
+    (pin "13")
+    (pin "14")
+    (pin "7")
   )
   (symbol (lib_id "Console-rescue:R") (at 186.69 83.82 0) (unit 1)
@@
       (effects (font (size 1.524 1.524)))
     )
-    (pin "10")
-    (pin "8")
-    (pin "9")
-  )
-  (symbol (lib_id "74xx:74LS32") (at 187.96 123.19 0) (unit 4)
-    (in_bom yes) (on_board yes)
-    (property "Reference" "U9" (id 0) (at 187.96 121.92 0)
-      (effects (font (size 1.524 1.524)))
-    )
-    (property "Value" "74LS32" (id 1) (at 187.96 124.46 0)
-      (effects (font (size 1.524 1.524)))
-    )
-    (property "Footprint" "Package_DIP:DIP-14_W7.62mm_Socket_LongPads" (id 2) (at 187.96 123.19 0)
-      (effects (font (size 1.524 1.524)) hide)
-    )
-    (property "Datasheet" "" (id 3) (at 187.96 123.19 0)
-      (effects (font (size 1.524 1.524)))
-    )
+    (pin "1")
+    (pin "2")
+    (pin "3")
+    (pin "4")
+    (pin "5")
+    (pin "6")
+    (pin "10")
+    (pin "8")
+    (pin "9")
     (pin "11")
     (pin "12")
     (pin "13")
+    (pin "14")
+    (pin "7")
+  )
+  (symbol (lib_id "74xx:74LS32") (at 187.96 123.19 0) (unit 4)
+    (in_bom yes) (on_board yes)
+    (property "Reference" "U9" (id 0) (at 187.96 121.92 0)
+      (effects (font (size 1.524 1.524)))
+    )
+    (property "Value" "74LS32" (id 1) (at 187.96 124.46 0)
+      (effects (font (size 1.524 1.524)))
+    )
+    (property "Footprint" "Package_DIP:DIP-14_W7.62mm_Socket_LongPads" (id 2) (at 187.96 123.19 0)
+      (effects (font (size 1.524 1.524)) hide)
+    )
+    (property "Datasheet" "" (id 3) (at 187.96 123.19 0)
+      (effects (font (size 1.524 1.524)))
+    )
+    (pin "1")
+    (pin "2")
+    (pin "3")
+    (pin "4")
+    (pin "5")
+    (pin "6")
+    (pin "10")
+    (pin "8")
+    (pin "9")
+    (pin "11")
+    (pin "12")
+    (pin "13")
+    (pin "14")
+    (pin "7")
   )
   (symbol (lib_id "74xx:74LS32") (at 172.72 128.27 0) (unit 1)
@@
     (pin "2")
     (pin "3")
+    (pin "4")
+    (pin "5")
+    (pin "6")
+    (pin "10")
+    (pin "8")
+    (pin "9")
+    (pin "11")
+    (pin "12")
+    (pin "13")
+    (pin "14")
+    (pin "7")
   )
   (symbol (lib_id "Console-rescue:R") (at 113.03 78.74 180) (unit 1)
@@
     (pin "1")
   )
-  (symbol (lib_id "74xx:74LS32") (at 160.02 153.67 0) (unit 1)
-    (in_bom yes) (on_board yes) (fields_autoplaced)
-    (property "Reference" "U7" (id 0) (at 160.02 144.78 0))
-    (property "Value" "74LS32" (id 1) (at 160.02 147.32 0))
-    (property "Footprint" "Package_DIP:DIP-14_W7.62mm_Socket_LongPads" (id 2) (at 160.02 153.67 0)
-      (effects (font (size 1.27 1.27)) hide)
-    )
-    (property "Datasheet" "http://www.ti.com/lit/gpn/sn74LS32" (id 3) (at 160.02 153.67 0)
-      (effects (font (size 1.27 1.27)) hide)
-    )
-    (pin "1")
-    (pin "2")
-    (pin "3")
-  )
-  (symbol (lib_id "74xx:74LS32") (at 143.51 165.1 0) (unit 4)
-    (in_bom yes) (on_board yes) (fields_autoplaced)
-    (property "Reference" "U7" (id 0) (at 143.51 156.21 0))
-    (property "Value" "74LS32" (id 1) (at 143.51 158.75 0))
-    (property "Footprint" "Package_DIP:DIP-14_W7.62mm_Socket_LongPads" (id 2) (at 143.51 165.1 0)
-      (effects (font (size 1.27 1.27)) hide)
-    )
-    (property "Datasheet" "http://www.ti.com/lit/gpn/sn74LS32" (id 3) (at 143.51 165.1 0)
-      (effects (font (size 1.27 1.27)) hide)
-    )
+  (symbol (lib_id "74xx:74LS08") (at 124.46 157.48 0) (unit 3)
+    (in_bom yes) (on_board yes)
+    (property "Reference" "U7" (id 0) (at 123.19 165.1 0))
+    (property "Value" "74LS08" (id 1) (at 123.19 162.56 0))
+    (property "Footprint" "Package_DIP:DIP-14_W7.62mm_Socket_LongPads" (id 2) (at 124.46 157.48 0)
+      (effects (font (size 1.27 1.27)) hide)
+    )
+    (property "Datasheet" "http://www.ti.com/lit/gpn/sn74LS08" (id 3) (at 124.46 157.48 0)
+      (effects (font (size 1.27 1.27)) hide)
+    )
+    (pin "1")
+    (pin "2")
+    (pin "3")
+    (pin "4")
+    (pin "5")
+    (pin "6")
+    (pin "10")
+    (pin "8")
+    (pin "9")
     (pin "11")
     (pin "12")
     (pin "13")
-  )
-  (symbol (lib_id "74xx:74LS32") (at 124.46 148.59 0) (unit 2)
+    (pin "14")
+    (pin "7")
+  )
+  (symbol (lib_id "74xx:74LS08") (at 160.02 153.67 0) (unit 1)
     (in_bom yes) (on_board yes) (fields_autoplaced)
-    (property "Reference" "U7" (id 0) (at 124.46 139.7 0))
-    (property "Value" "74LS32" (id 1) (at 124.46 142.24 0))
-    (property "Footprint" "Package_DIP:DIP-14_W7.62mm_Socket_LongPads" (id 2) (at 124.46 148.59 0)
-      (effects (font (size 1.27 1.27)) hide)
-    )
-    (property "Datasheet" "http://www.ti.com/lit/gpn/sn74LS32" (id 3) (at 124.46 148.59 0)
-      (effects (font (size 1.27 1.27)) hide)
-    )
-    (pin "4")
-    (pin "5")
-    (pin "6")
+    (property "Reference" "U7" (id 0) (at 160.02 146.1602 0))
+    (property "Value" "74LS08" (id 1) (at 160.02 148.6971 0))
+    (property "Footprint" "Package_DIP:DIP-14_W7.62mm_Socket_LongPads" (id 2) (at 160.02 153.67 0)
+      (effects (font (size 1.27 1.27)) hide)
+    )
+    (property "Datasheet" "http://www.ti.com/lit/gpn/sn74LS08" (id 3) (at 160.02 153.67 0)
+      (effects (font (size 1.27 1.27)) hide)
+    )
+    (pin "1")
+    (pin "2")
+    (pin "3")
+    (pin "4")
+    (pin "5")
+    (pin "6")
+    (pin "10")
+    (pin "8")
+    (pin "9")
+    (pin "11")
+    (pin "12")
+    (pin "13")
+    (pin "14")
+    (pin "7")
   )
   (symbol (lib_id "Device:R") (at 105.41 172.72 0) (unit 1)
@@
     (pin "1")
     (pin "2")
+  )
+  (symbol (lib_id "74xx:74LS08") (at 124.46 148.59 0) (unit 2)
+    (in_bom yes) (on_board yes) (fields_autoplaced)
+    (property "Reference" "U7" (id 0) (at 124.46 141.0802 0))
+    (property "Value" "74LS08" (id 1) (at 124.46 143.6171 0))
+    (property "Footprint" "Package_DIP:DIP-14_W7.62mm_Socket_LongPads" (id 2) (at 124.46 148.59 0)
+      (effects (font (size 1.27 1.27)) hide)
+    )
+    (property "Datasheet" "http://www.ti.com/lit/gpn/sn74LS08" (id 3) (at 124.46 148.59 0)
+      (effects (font (size 1.27 1.27)) hide)
+    )
+    (pin "1")
+    (pin "2")
+    (pin "3")
+    (pin "4")
+    (pin "5")
+    (pin "6")
+    (pin "10")
+    (pin "8")
+    (pin "9")
+    (pin "11")
+    (pin "12")
+    (pin "13")
+    (pin "14")
+    (pin "7")
   )
   (symbol (lib_id "Device:R") (at 101.6 172.72 0) (unit 1)
@@
     (pin "2")
   )
-  (symbol (lib_id "74xx:74LS32") (at 124.46 157.48 0) (unit 3)
-    (in_bom yes) (on_board yes)
-    (property "Reference" "U7" (id 0) (at 124.46 165.1 0))
-    (property "Value" "74LS32" (id 1) (at 124.46 162.56 0))
-    (property "Footprint" "Package_DIP:DIP-14_W7.62mm_Socket_LongPads" (id 2) (at 124.46 157.48 0)
-      (effects (font (size 1.27 1.27)) hide)
-    )
-    (property "Datasheet" "http://www.ti.com/lit/gpn/sn74LS32" (id 3) (at 124.46 157.48 0)
-      (effects (font (size 1.27 1.27)) hide)
-    )
-    (pin "10")
-    (pin "8")
-    (pin "9")
+  (symbol (lib_id "74xx:74LS08") (at 143.51 165.1 0) (unit 4)
+    (in_bom yes) (on_board yes) (fields_autoplaced)
+    (property "Reference" "U7" (id 0) (at 143.51 157.5902 0))
+    (property "Value" "74LS08" (id 1) (at 143.51 160.1271 0))
+    (property "Footprint" "Package_DIP:DIP-14_W7.62mm_Socket_LongPads" (id 2) (at 143.51 165.1 0)
+      (effects (font (size 1.27 1.27)) hide)
+    )
+    (property "Datasheet" "http://www.ti.com/lit/gpn/sn74LS08" (id 3) (at 143.51 165.1 0)
+      (effects (font (size 1.27 1.27)) hide)
+    )
+    (pin "1")
+    (pin "2")
+    (pin "3")
+    (pin "4")
+    (pin "5")
+    (pin "6")
+    (pin "10")
+    (pin "8")
+    (pin "9")
+    (pin "11")
+    (pin "12")
+    (pin "13")
+    (pin "14")
+    (pin "7")
   )
 )

Commit message: hardware updates
Parts:
- removed R18: 1kΩ, Resistor_THT:R_Axial_DIN0207_L6.3mm_D2.5mm_P7.62mm_Horizontal, symbol Console-rescue:R
- SW1: footprint Package_DIP:DIP-10_W10.16mm_LongPads -> Package_DIP:DIP-10_W7.62mm_Socket_LongPads
Connections:
- net ~{ROM}: now also U5.15 (O0)
Changed lines of the file:
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@@
     (stroke (width 0) (type default) (color 0 0 0 0))
   )
-  (wire (pts (xy 146.05 105.41) (xy 111.76 105.41))
+  (wire (pts (xy 111.76 105.41) (xy 153.67 105.41))
     (stroke (width 0) (type default) (color 0 0 0 0))
   )
@@
     )
     (pin "1")
-  )
-  (symbol (lib_id "Console-rescue:R") (at 149.86 105.41 270) (unit 1)
-    (in_bom yes) (on_board yes)
-    (property "Reference" "R18" (id 0) (at 149.86 105.41 90))
-    (property "Value" "1kΩ" (id 1) (at 149.86 102.87 90))
-    (property "Footprint" "Resistor_THT:R_Axial_DIN0207_L6.3mm_D2.5mm_P7.62mm_Horizontal" (id 2) (at 149.86 103.632 90)
-      (effects (font (size 0.762 0.762)) hide)
-    )
-    (property "Datasheet" "" (id 3) (at 149.86 105.41 0)
-      (effects (font (size 0.762 0.762)))
-    )
-    (pin "1")
-    (pin "2")
   )
   (symbol (lib_id "74xx:74LS32") (at 212.09 120.65 0) (unit 3)
@@
     (property "Reference" "SW1" (id 0) (at 80.01 143.51 0))
     (property "Value" "RAM Size" (id 1) (at 80.01 146.05 0))
-    (property "Footprint" "Package_DIP:DIP-10_W10.16mm_LongPads" (id 2) (at 80.01 156.21 0)
-      (effects (font (size 1.27 1.27)) hide)
-    )
+    (property "Footprint" "Package_DIP:DIP-10_W7.62mm_Socket_LongPads" (id 2) (at 80.01 156.21 0)
+      (effects (font (size 1.27 1.27)) hide)
+    )

Commit message: hardware updates
Parts:
- renumbered R19 to R18
Changed lines of the file:
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@@
   (symbol (lib_id "Console-rescue:R") (at 186.69 83.82 0) (unit 1)
     (in_bom yes) (on_board yes)
-    (property "Reference" "R19" (id 0) (at 186.69 83.82 90))
+    (property "Reference" "R18" (id 0) (at 186.69 83.82 90))
     (property "Value" "1kΩ" (id 1) (at 184.15 83.82 90))
     (property "Footprint" "Resistor_THT:R_Axial_DIN0207_L6.3mm_D2.5mm_P7.62mm_Horizontal" (id 2) (at 184.912 83.82 90)

Commit message: PCB cleanup
Parts:
- R11, R17, R18: symbol Console-rescue:R -> Device:R
Other:
- moved on the sheet: C12
