File: mainboard/CPU.kicad_sch (KiCad schematic)
At the start: 31 parts, among them J1 Reset, U1 TIM9904, U2 TMS9900, U3 74LS04, U4 74LS32, Y1 48.000 MHz

Commit message: PCB routed
Parts:
- C10, C3, C5: footprint Capacitor_THT:C_Rect_L7.0mm_W2.0mm_P5.00mm -> Capacitor_THT:CP_Radial_D7.5mm_P2.50mm
- J1: footprint (none) -> Connector_PinHeader_2.54mm:PinHeader_1x02_P2.54mm_Vertical
- U1: footprint Package_DIP:DIP-20_W7.62mm_LongPads -> Package_DIP:DIP-20_W7.62mm_Socket_LongPads
- U2: footprint (none) -> Package_DIP:DIP-64_W22.86mm_Socket_LongPads
- U3, U4: footprint Package_DIP:DIP-14_W7.62mm_LongPads -> Package_DIP:DIP-14_W7.62mm_Socket_LongPads
- Y1: footprint (none) -> Crystal:Crystal_HC49-U_Vertical
Changed lines of the file:
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@@
       (effects (font (size 1.524 1.524)))
     )
-    (property "Footprint" "" (id 2) (at 157.48 116.84 0)
+    (property "Footprint" "Package_DIP:DIP-64_W22.86mm_Socket_LongPads" (id 2) (at 157.48 116.84 0)
       (effects (font (size 1.524 1.524)) hide)
     )
@@
       (effects (font (size 1.524 1.524)))
     )
-    (property "Footprint" "Package_DIP:DIP-20_W7.62mm_LongPads" (id 2) (at 111.76 74.93 0)
+    (property "Footprint" "Package_DIP:DIP-20_W7.62mm_Socket_LongPads" (id 2) (at 111.76 74.93 0)
       (effects (font (size 1.524 1.524)) hide)
     )
@@
     (property "Reference" "Y1" (id 0) (at 88.9 73.66 0))
     (property "Value" "48.000 MHz" (id 1) (at 88.9 81.28 0))
-    (property "Footprint" "" (id 2) (at 88.9 77.47 0)
+    (property "Footprint" "Crystal:Crystal_HC49-U_Vertical" (id 2) (at 88.9 77.47 0)
       (effects (font (size 1.524 1.524)) hide)
     )
@@
       (effects (font (size 1.27 1.27)) (justify left))
     )
-    (property "Footprint" "Capacitor_THT:C_Rect_L7.0mm_W2.0mm_P5.00mm" (id 2) (at 107.95 33.02 0)
+    (property "Footprint" "Capacitor_THT:CP_Radial_D7.5mm_P2.50mm" (id 2) (at 107.95 33.02 0)
       (effects (font (size 1.524 1.524)) hide)
     )
@@
       (effects (font (size 1.27 1.27)) (justify left))
     )
-    (property "Footprint" "Capacitor_THT:C_Rect_L7.0mm_W2.0mm_P5.00mm" (id 2) (at 78.74 33.02 0)
+    (property "Footprint" "Capacitor_THT:CP_Radial_D7.5mm_P2.50mm" (id 2) (at 78.74 33.02 0)
       (effects (font (size 1.524 1.524)) hide)
     )
@@
       (effects (font (size 1.524 1.524)))
     )
-    (property "Footprint" "Package_DIP:DIP-14_W7.62mm_LongPads" (id 2) (at 194.31 113.03 0)
+    (property "Footprint" "Package_DIP:DIP-14_W7.62mm_Socket_LongPads" (id 2) (at 194.31 113.03 0)
       (effects (font (size 1.524 1.524)) hide)
     )
@@
       (effects (font (size 1.27 1.27)) (justify left))
     )
-    (property "Footprint" "Capacitor_THT:C_Rect_L7.0mm_W2.0mm_P5.00mm" (id 2) (at 187.96 52.07 0)
+    (property "Footprint" "Capacitor_THT:CP_Radial_D7.5mm_P2.50mm" (id 2) (at 187.96 52.07 0)
       (effects (font (size 1.524 1.524)) hide)
     )
@@
       (effects (font (size 1.524 1.524)))
     )
-    (property "Footprint" "Package_DIP:DIP-14_W7.62mm_LongPads" (id 2) (at 209.55 104.14 0)
+    (property "Footprint" "Package_DIP:DIP-14_W7.62mm_Socket_LongPads" (id 2) (at 209.55 104.14 0)
       (effects (font (size 1.524 1.524)) hide)
     )
@@
     (property "Reference" "J1" (id 0) (at 81.915 107.95 0))
     (property "Value" "Reset" (id 1) (at 81.915 110.49 0))
-    (property "Footprint" "" (id 2) (at 81.28 113.03 0)
-      (effects (font (size 1.27 1.27)) hide)
-    )
+    (property "Footprint" "Connector_PinHeader_2.54mm:PinHeader_1x02_P2.54mm_Vertical" (id 2) (at 81.28 113.03 0)
+      (effects (font (size 1.27 1.27)) hide)
+    )

Commit message: unicorn work
Changed lines of the file:
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@@
   (title_block
     (title "TI-99/22")
-    (date "2022-06-23")
-    (rev "0.75")
+    (date "2022-10-11")
+    (rev "0.76")
     (company "Dan Werner - https://github.com/danwerner21/ti99_22")
     (comment 1 "CPU and Clock Generator")
@@
     (in_bom yes) (on_board yes)
     (property "Reference" "R2" (id 0) (at 88.9 85.09 90))
-    (property "Value" "1kΩ" (id 1) (at 92.71 83.82 90)
+    (property "Value" "1kΩ" (id 1) (at 87.63 87.63 90)
       (effects (font (size 1.27 1.27)) (justify left))
     )
@@
       (effects (font (size 1.27 1.27)) (justify left))
     )
-    (property "Value" "6.8µH" (id 1) (at 119.126 52.578 0)
+    (property "Value" "6.8µH" (id 1) (at 120.65 54.61 90)
       (effects (font (size 1.27 1.27)) (justify left))
     )
@@
     (pin "1")
     (pin "2")
+    (pin "3")
+    (pin "4")
+    (pin "5")
+    (pin "6")
+    (pin "8")
+    (pin "9")
+    (pin "10")
+    (pin "11")
+    (pin "12")
+    (pin "13")
+    (pin "14")
+    (pin "7")
   )
   (symbol (lib_id "TI-Customs:C_Small") (at 128.27 53.34 90) (unit 1)
@@
       (effects (font (size 1.27 1.27)) (justify left))
     )
-    (property "Value" "1µF" (id 1) (at 130.81 52.705 0)
+    (property "Value" "1µF" (id 1) (at 134.62 52.07 90)
       (effects (font (size 1.27 1.27)) (justify left))
     )
@@
   (symbol (lib_id "TI-Customs:C_Small") (at 106.68 48.26 270) (unit 1)
     (in_bom yes) (on_board yes)
-    (property "Reference" "C4" (id 0) (at 109.22 48.895 0)
-      (effects (font (size 1.27 1.27)) (justify left))
-    )
-    (property "Value" "0.1µF" (id 1) (at 104.14 48.895 0)
+    (property "Reference" "C4" (id 0) (at 105.41 50.8 90)
+      (effects (font (size 1.27 1.27)) (justify left))
+    )
+    (property "Value" "0.1µF" (id 1) (at 104.14 45.72 90)
       (effects (font (size 1.27 1.27)) (justify left))
     )
@@
     (in_bom yes) (on_board yes)
     (property "Reference" "R9" (id 0) (at 184.15 90.17 90))
-    (property "Value" "1kΩ" (id 1) (at 190.5 87.63 90)
+    (property "Value" "1kΩ" (id 1) (at 185.42 92.71 90)
       (effects (font (size 1.27 1.27)) (justify right))
     )
@@
     (pin "2")
     (pin "3")
+    (pin "4")
+    (pin "5")
+    (pin "6")
+    (pin "10")
+    (pin "8")
+    (pin "9")
+    (pin "11")
+    (pin "12")
+    (pin "13")
+    (pin "14")
+    (pin "7")
   )
   (symbol (lib_id "Console-rescue:GND") (at 201.93 101.6 270) (unit 1)

Commit message: PCB cleanup
Parts:
- C1, C11, C2, C4, C6, C7, C8, C9: symbol TI-Customs:C_Small -> Device:C
- C10: symbol Device:CP_Small -> Device:C_Polarized_Small
- C3, C5: symbol Device:CP -> Device:C_Polarized
- L1, L2, L3, L4: symbol Console-rescue:L_Small -> Device:L_Small
- R1, R10, R2, R3, R4, R5, R6, R7, R8, R9: symbol Console-rescue:R -> Device:R
- U1: symbol TI-Customs:TIM9904 -> Werner_custom:TIM9904
- U2: symbol TI-Customs:TMS9900 -> Werner_custom:TMS9900
- Y1: symbol Console-rescue:Crystal -> Device:Crystal
Other:
- moved on the sheet: C4, C7, C8

Commit message: PCB power fix
Parts:
- removed L4: 6.8µH, Resistor_THT:R_Axial_DIN0207_L6.3mm_D2.5mm_P7.62mm_Horizontal, symbol Device:L_Small
Connections:
- net +5V: now also C11.1, R10.1, U2.2 (VCC)
Changed lines of the file:
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@@
   (title_block
     (title "TI-99/22")
-    (date "2022-10-11")
-    (rev "0.76")
+    (date "2022-12-25")
+    (rev "0.95")
     (company "Dan Werner - https://github.com/danwerner21/ti99_22")
     (comment 1 "CPU and Clock Generator")
@@
   (junction (at 158.75 163.83) (diameter 0) (color 0 0 0 0)
   )
-  (junction (at 168.402 64.77) (diameter 0) (color 0 0 0 0)
-  )
   (junction (at 123.19 53.34) (diameter 0) (color 0 0 0 0)
   )
@@
   )
   (junction (at 175.26 59.69) (diameter 0) (color 0 0 0 0)
+  )
+  (junction (at 158.75 64.77) (diameter 0) (color 0 0 0 0)
   )
   (junction (at 109.22 48.26) (diameter 0) (color 0 0 0 0)
@@
     (stroke (width 0) (type default) (color 0 0 0 0))
   )
+  (wire (pts (xy 158.75 64.77) (xy 158.75 73.66))
+    (stroke (width 0) (type default) (color 0 0 0 0))
+  )
   (wire (pts (xy 109.22 48.26) (xy 146.05 48.26))
     (stroke (width 0) (type default) (color 0 0 0 0))
@@
     (stroke (width 0) (type default) (color 0 0 0 0))
   )
-  (wire (pts (xy 175.26 52.07) (xy 175.26 53.34))
-    (stroke (width 0) (type default) (color 0 0 0 0))
-  )
   (wire (pts (xy 73.66 85.09) (xy 85.09 85.09))
     (stroke (width 0) (type default) (color 0 0 0 0))
@@
     (stroke (width 0) (type default) (color 0 0 0 0))
   )
+  (wire (pts (xy 158.75 64.77) (xy 175.26 64.77))
+    (stroke (width 0) (type default) (color 0 0 0 0))
+  )
   (wire (pts (xy 77.47 66.04) (xy 83.82 66.04))
     (stroke (width 0) (type default) (color 0 0 0 0))
@@
     (stroke (width 0) (type default) (color 0 0 0 0))
   )
-  (wire (pts (xy 168.402 64.77) (xy 175.26 64.77))
-    (stroke (width 0) (type default) (color 0 0 0 0))
-  )
   (wire (pts (xy 185.42 52.07) (xy 175.26 52.07))
     (stroke (width 0) (type default) (color 0 0 0 0))
@@
     (stroke (width 0) (type default) (color 0 0 0 0))
   )
-  (wire (pts (xy 158.75 52.07) (xy 175.26 52.07))
-    (stroke (width 0) (type default) (color 0 0 0 0))
-  )
   (wire (pts (xy 175.26 59.69) (xy 184.15 59.69))
     (stroke (width 0) (type default) (color 0 0 0 0))
@@
     (stroke (width 0) (type default) (color 0 0 0 0))
   )
-  (wire (pts (xy 175.26 58.42) (xy 175.26 59.69))
+  (wire (pts (xy 175.26 52.07) (xy 175.26 59.69))
     (stroke (width 0) (type default) (color 0 0 0 0))
   )
@@
     (stroke (width 0) (type default) (color 0 0 0 0))
   )
-  (wire (pts (xy 156.21 64.77) (xy 168.402 64.77))
+  (wire (pts (xy 156.21 64.77) (xy 158.75 64.77))
     (stroke (width 0) (type default) (color 0 0 0 0))
   )
   (wire (pts (xy 149.86 160.02) (xy 149.86 163.83))
-    (stroke (width 0) (type default) (color 0 0 0 0))
-  )
-  (wire (pts (xy 158.75 52.07) (xy 158.75 73.66))
     (stroke (width 0) (type default) (color 0 0 0 0))
   )
@@
     (pin "1")
   )
-  (symbol (lib_id "Device:L_Small") (at 175.26 55.88 0) (unit 1)
-    (in_bom yes) (on_board yes)
-    (property "Reference" "L4" (id 0) (at 168.91 54.61 0)
-      (effects (font (size 1.27 1.27)) (justify left))
-    )
-    (property "Value" "6.8µH" (id 1) (at 168.91 57.15 0)
-      (effects (font (size 1.27 1.27)) (justify left))
-    )
-    (property "Footprint" "Resistor_THT:R_Axial_DIN0207_L6.3mm_D2.5mm_P7.62mm_Horizontal" (id 2) (at 175.26 55.88 0)
-      (effects (font (size 1.27 1.27)) hide)
-    )
-    (property "Datasheet" "~" (id 3) (at 175.26 55.88 0)
-      (effects (font (size 1.27 1.27)) hide)
-    )
-    (pin "1")
-    (pin "2")
-  )
   (symbol (lib_id "power:+5V") (at 175.26 44.45 0) (unit 1)
     (in_bom yes) (on_board yes)
@@
       (effects (font (size 1.27 1.27)) hide)
     )
-    (pin "1")
-  )
-  (symbol (lib_id "power:PWR_FLAG") (at 168.402 64.77 0) (unit 1)
-    (in_bom yes) (on_board yes) (fields_autoplaced)
-    (property "Reference" "#FLG0101" (id 0) (at 168.402 62.865 0)
-      (effects (font (size 1.27 1.27)) hide)
-    )
-    (property "Value" "PWR_FLAG" (id 1) (at 168.402 61.1942 0))
-    (property "Footprint" "" (id 2) (at 168.402 64.77 0)
-      (effects (font (size 1.27 1.27)) hide)
-    )
-    (property "Datasheet" "~" (id 3) (at 168.402 64.77 0)
-      (effects (font (size 1.27 1.27)) hide)
-    )

Commit message: PCB rework
Parts:
- removed L2, L3: 6.8µH, Resistor_THT:R_Axial_DIN0207_L6.3mm_D2.5mm_P7.62mm_Horizontal, symbol Device:L_Small
- L1: footprint Resistor_THT:R_Axial_DIN0207_L6.3mm_D2.5mm_P7.62mm_Horizontal -> Resistor_THT:R_Axial_DIN0207_L6.3mm_D2.5mm_P15.24mm_Horizontal
Connections:
- net +12V: now also C4.1, C7.1, U1.13 (VDD), U2.27 (VDD)
- net +5V: now also C1.1, R2.2, U1.20 (VCC)
Changed lines of the file:
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@@
   (title_block
     (title "TI-99/22")
-    (date "2022-12-25")
+    (date "2022-12-26")
     (rev "0.95")
     (company "Dan Werner - https://github.com/danwerner21/ti99_22")
-    (comment 1 "CPU and Clock Generator")
+    (comment 1 "Schematic for Keyboard, Joystick and Cassette port.")
     (comment 3 "was based on the HackMac KiCAD Design")
     (comment 4 "Based Robert Krenicki's design which")
@@
   (junction (at 83.82 66.04) (diameter 0) (color 0 0 0 0)
   )
-  (junction (at 162.56 48.26) (diameter 0) (color 0 0 0 0)
-  )
   (junction (at 114.3 36.83) (diameter 0) (color 0 0 0 0)
   )
@@
     (stroke (width 0) (type default) (color 0 0 0 0))
   )
-  (wire (pts (xy 149.86 40.64) (xy 149.86 38.1))
+  (wire (pts (xy 149.86 38.1) (xy 149.86 48.26))
     (stroke (width 0) (type default) (color 0 0 0 0))
   )
@@
     (stroke (width 0) (type default) (color 0 0 0 0))
   )
-  (wire (pts (xy 114.3 53.34) (xy 115.57 53.34))
-    (stroke (width 0) (type default) (color 0 0 0 0))
-  )
   (wire (pts (xy 191.77 59.69) (xy 193.04 59.69))
     (stroke (width 0) (type default) (color 0 0 0 0))
@@
     (stroke (width 0) (type default) (color 0 0 0 0))
   )
-  (wire (pts (xy 120.65 53.34) (xy 123.19 53.34))
+  (wire (pts (xy 114.3 53.34) (xy 123.19 53.34))
     (stroke (width 0) (type default) (color 0 0 0 0))
   )
@@
   )
   (wire (pts (xy 77.47 66.04) (xy 83.82 66.04))
-    (stroke (width 0) (type default) (color 0 0 0 0))
-  )
-  (wire (pts (xy 149.86 48.26) (xy 149.86 45.72))
     (stroke (width 0) (type default) (color 0 0 0 0))
   )
@@
     (pin "1")
   )
-  (symbol (lib_id "Device:L_Small") (at 118.11 53.34 90) (unit 1)
-    (in_bom yes) (on_board yes)
-    (property "Reference" "L2" (id 0) (at 117.094 52.578 0)
-      (effects (font (size 1.27 1.27)) (justify left))
-    )
-    (property "Value" "6.8µH" (id 1) (at 120.65 54.61 90)
-      (effects (font (size 1.27 1.27)) (justify left))
-    )
-    (property "Footprint" "Resistor_THT:R_Axial_DIN0207_L6.3mm_D2.5mm_P7.62mm_Horizontal" (id 2) (at 118.11 53.34 0)
-      (effects (font (size 1.27 1.27)) hide)
-    )
-    (property "Datasheet" "~" (id 3) (at 118.11 53.34 0)
-      (effects (font (size 1.27 1.27)) hide)
-    )
-    (pin "1")
-    (pin "2")
-  )
   (symbol (lib_id "Device:C") (at 69.85 57.15 0) (unit 1)
     (in_bom yes) (on_board yes)
@@
     (pin "1")
   )
-  (symbol (lib_id "Device:L_Small") (at 149.86 43.18 0) (unit 1)
-    (in_bom yes) (on_board yes)
-    (property "Reference" "L3" (id 0) (at 150.622 42.164 0)
-      (effects (font (size 1.27 1.27)) (justify left))
-    )
-    (property "Value" "6.8µH" (id 1) (at 150.622 44.196 0)
-      (effects (font (size 1.27 1.27)) (justify left))
-    )
-    (property "Footprint" "Resistor_THT:R_Axial_DIN0207_L6.3mm_D2.5mm_P7.62mm_Horizontal" (id 2) (at 149.86 43.18 0)
-      (effects (font (size 1.27 1.27)) hide)
-    )
-    (property "Datasheet" "~" (id 3) (at 149.86 43.18 0)
-      (effects (font (size 1.27 1.27)) hide)
-    )
-    (pin "1")
-    (pin "2")
-  )
   (symbol (lib_id "Device:L_Small") (at 83.82 60.96 0) (unit 1)
     (in_bom yes) (on_board yes)
@@
       (effects (font (size 1.27 1.27)) (justify left))
     )
-    (property "Footprint" "Resistor_THT:R_Axial_DIN0207_L6.3mm_D2.5mm_P7.62mm_Horizontal" (id 2) (at 83.82 60.96 0)
+    (property "Footprint" "Resistor_THT:R_Axial_DIN0207_L6.3mm_D2.5mm_P15.24mm_Horizontal" (id 2) (at 83.82 60.96 0)
       (effects (font (size 1.27 1.27)) hide)
     )
@@
       (effects (font (size 1.27 1.27)) hide)
     )
-    (pin "1")
-  )
-  (symbol (lib_id "power:PWR_FLAG") (at 114.3 53.34 0) (unit 1)
-    (in_bom yes) (on_board yes) (fields_autoplaced)
-    (property "Reference" "#FLG0103" (id 0) (at 114.3 51.435 0)
-      (effects (font (size 1.27 1.27)) hide)
-    )
-    (property "Value" "PWR_FLAG" (id 1) (at 114.3 49.7642 0))
-    (property "Footprint" "" (id 2) (at 114.3 53.34 0)
-      (effects (font (size 1.27 1.27)) hide)
-    )
-    (property "Datasheet" "~" (id 3) (at 114.3 53.34 0)
-      (effects (font (size 1.27 1.27)) hide)
-    )
-    (pin "1")
-  )
-  (symbol (lib_id "power:PWR_FLAG") (at 162.56 48.26 0) (unit 1)
-    (in_bom yes) (on_board yes) (fields_autoplaced)
-    (property "Reference" "#FLG0102" (id 0) (at 162.56 46.355 0)
-      (effects (font (size 1.27 1.27)) hide)
-    )
-    (property "Value" "PWR_FLAG" (id 1) (at 162.56 44.6842 0))
-    (property "Footprint" "" (id 2) (at 162.56 48.26 0)
-      (effects (font (size 1.27 1.27)) hide)
-    )
-    (property "Datasheet" "~" (id 3) (at 162.56 48.26 0)
-      (effects (font (size 1.27 1.27)) hide)
-    )
