File: mainboard/Cassette.kicad_sch (KiCad schematic)
At the start: 43 parts, among them J18 Cassette, Q3 TIS92, Q4 TIS92, U46 RC4558, U47 74LS06, U48 TIL119, U49 TIL119

Commit message: PCB 0.96
Parts:
- J18: footprint Connector_Dsub:DSUB-9_Female_Horizontal_P2.77x2.84mm_EdgePinOffset4.94mm_Housed_MountingHolesOffset7.48mm -> Connector_Dsub:DSUB-9_Male_Horizontal_P2.77x2.84mm_EdgePinOffset4.94mm_Housed_MountingHolesOffset7.48mm
Changed lines of the file:
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@@
   (title_block
     (title "TI-99/22")
-    (date "2022-12-26")
-    (rev "0.95")
+    (date "2023-01-21")
+    (rev "0.96")
     (company "Dan Werner - https://github.com/danwerner21/ti99_22")
     (comment 1 "Schematic for Keyboard, Joystick and Cassette port.")
@@
       (effects (font (size 1.778 1.778)))
     )
-    (property "Footprint" "Connector_Dsub:DSUB-9_Female_Horizontal_P2.77x2.84mm_EdgePinOffset4.94mm_Housed_MountingHolesOffset7.48mm" (id 2) (at 215.138 60.96 0)
+    (property "Footprint" "Connector_Dsub:DSUB-9_Male_Horizontal_P2.77x2.84mm_EdgePinOffset4.94mm_Housed_MountingHolesOffset7.48mm" (id 2) (at 215.138 60.96 0)
       (effects (font (size 1.524 1.524)) hide)
     )
