File: mainboard/GROM-Logic.kicad_sch (KiCad schematic)
At the start: 17 parts, among them J4 UNICORN PORT, Q1 TIS92, U15 74LS04, U20 74LS04, U23 TMC0430, U24 TMC0430, U25 TMC0430, U6 74LS03

Commit message: PCB rework
Parts:
- renumbered C51 to C52, U20 to U22, U23 to U26, U24 to U27, U25 to U28
Changed lines of the file:
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@@
   (title_block
     (title "TI-99/22")
-    (date "2022-10-11")
-    (rev "0.76")
+    (date "2022-12-26")
+    (rev "0.95")
     (company "Dan Werner - https://github.com/danwerner21/ti99_22")
-    (comment 1 "GROM with Logic")
+    (comment 1 "Schematic for Keyboard, Joystick and Cassette port.")
     (comment 3 "was based on the HackMac KiCAD Design")
     (comment 4 "Based Robert Krenicki's design which")
@@
   (symbol (lib_id "power:-5V") (at 40.64 85.09 180) (unit 1)
     (in_bom yes) (on_board yes)
-    (property "Reference" "#PWR070" (id 0) (at 40.64 87.63 0)
+    (property "Reference" "#PWR072" (id 0) (at 40.64 87.63 0)
       (effects (font (size 1.27 1.27)) hide)
     )
@@
   (symbol (lib_id "power:-5V") (at 86.36 85.09 180) (unit 1)
     (in_bom yes) (on_board yes)
-    (property "Reference" "#PWR078" (id 0) (at 86.36 87.63 0)
+    (property "Reference" "#PWR080" (id 0) (at 86.36 87.63 0)
       (effects (font (size 1.27 1.27)) hide)
     )
@@
   (symbol (lib_id "power:-5V") (at 132.08 85.09 180) (unit 1)
     (in_bom yes) (on_board yes)
-    (property "Reference" "#PWR083" (id 0) (at 132.08 87.63 0)
+    (property "Reference" "#PWR085" (id 0) (at 132.08 87.63 0)
       (effects (font (size 1.27 1.27)) hide)
     )
@@
   (symbol (lib_id "Device:C") (at 44.45 24.13 90) (unit 1)
     (in_bom yes) (on_board yes)
-    (property "Reference" "C51" (id 0) (at 49.53 26.67 90)
+    (property "Reference" "C52" (id 0) (at 49.53 26.67 90)
       (effects (font (size 1.27 1.27)) (justify left))
     )
@@
   (symbol (lib_id "power:GND") (at 48.26 24.13 90) (unit 1)
     (in_bom yes) (on_board yes)
-    (property "Reference" "#PWR073" (id 0) (at 54.61 24.13 0)
+    (property "Reference" "#PWR075" (id 0) (at 54.61 24.13 0)
       (effects (font (size 1.27 1.27)) hide)
     )
@@
   (symbol (lib_id "power:+5V") (at 68.58 124.46 0) (unit 1)
     (in_bom yes) (on_board yes)
-    (property "Reference" "#PWR076" (id 0) (at 68.58 128.27 0)
+    (property "Reference" "#PWR078" (id 0) (at 68.58 128.27 0)
       (effects (font (size 1.27 1.27)) hide)
     )
@@
   (symbol (lib_id "74xx:74LS04") (at 41.91 124.46 0) (unit 1)
     (in_bom yes) (on_board yes)
-    (property "Reference" "U20" (id 0) (at 46.863 121.539 0)
+    (property "Reference" "U22" (id 0) (at 46.863 121.539 0)
       (effects (font (size 1.524 1.524)))
     )
@@
   (symbol (lib_id "power:+12V") (at 46.99 158.75 0) (unit 1)
     (in_bom yes) (on_board yes)
-    (property "Reference" "#PWR071" (id 0) (at 46.99 162.56 0)
+    (property "Reference" "#PWR073" (id 0) (at 46.99 162.56 0)
       (effects (font (size 1.27 1.27)) hide)
     )
@@
   (symbol (lib_id "power:GND") (at 46.99 190.5 0) (unit 1)
     (in_bom yes) (on_board yes)
-    (property "Reference" "#PWR072" (id 0) (at 46.99 196.85 0)
+    (property "Reference" "#PWR074" (id 0) (at 46.99 196.85 0)
       (effects (font (size 1.27 1.27)) hide)
     )
@@
   (symbol (lib_id "power:GND") (at 60.96 173.99 270) (unit 1)
     (in_bom yes) (on_board yes)
-    (property "Reference" "#PWR075" (id 0) (at 54.61 173.99 0)
+    (property "Reference" "#PWR077" (id 0) (at 54.61 173.99 0)
       (effects (font (size 1.27 1.27)) hide)
     )
@@
   (symbol (lib_id "power:+5V") (at 60.96 149.86 0) (unit 1)
     (in_bom yes) (on_board yes)
-    (property "Reference" "#PWR074" (id 0) (at 60.96 153.67 0)
+    (property "Reference" "#PWR076" (id 0) (at 60.96 153.67 0)
       (effects (font (size 1.27 1.27)) hide)
     )
@@
   (symbol (lib_id "74xx:74LS04") (at 43.18 137.16 180) (unit 6)
     (in_bom yes) (on_board yes)
-    (property "Reference" "U20" (id 0) (at 38.227 140.081 0)
+    (property "Reference" "U22" (id 0) (at 38.227 140.081 0)
       (effects (font (size 1.524 1.524)))
     )
@@
   (symbol (lib_id "power:+5V") (at 114.3 166.37 90) (unit 1)
     (in_bom yes) (on_board yes)
-    (property "Reference" "#PWR081" (id 0) (at 118.11 166.37 0)
+    (property "Reference" "#PWR083" (id 0) (at 118.11 166.37 0)
       (effects (font (size 1.27 1.27)) hide)
     )
@@
   (symbol (lib_id "power:+5V") (at 86.36 24.13 0) (unit 1)
     (in_bom yes) (on_board yes) (fields_autoplaced)
-    (property "Reference" "#PWR077" (id 0) (at 86.36 27.94 0)
+    (property "Reference" "#PWR079" (id 0) (at 86.36 27.94 0)
       (effects (font (size 1.27 1.27)) hide)
     )
@@
   (symbol (lib_id "Werner_custom:TMC0430") (at 138.43 57.15 0) (unit 1)
     (in_bom yes) (on_board yes)
-    (property "Reference" "U25" (id 0) (at 144.78 27.94 0)
+    (property "Reference" "U28" (id 0) (at 144.78 27.94 0)
       (effects (font (size 1.27 1.27)) (justify left))
     )
@@
   (symbol (lib_id "power:GND") (at 109.22 168.91 0) (unit 1)
     (in_bom yes) (on_board yes)
-    (property "Reference" "#PWR080" (id 0) (at 109.22 175.26 0)
+    (property "Reference" "#PWR082" (id 0) (at 109.22 175.26 0)
       (effects (font (size 1.27 1.27)) hide)
     )
@@
   (symbol (lib_id "power:+5V") (at 40.64 24.13 0) (unit 1)
     (in_bom yes) (on_board yes) (fields_autoplaced)
-    (property "Reference" "#PWR069" (id 0) (at 40.64 27.94 0)
+    (property "Reference" "#PWR071" (id 0) (at 40.64 27.94 0)
       (effects (font (size 1.27 1.27)) hide)
     )
@@
   (symbol (lib_id "power:+5V") (at 132.08 24.13 0) (unit 1)
     (in_bom yes) (on_board yes) (fields_autoplaced)
-    (property "Reference" "#PWR082" (id 0) (at 132.08 27.94 0)
+    (property "Reference" "#PWR084" (id 0) (at 132.08 27.94 0)
       (effects (font (size 1.27 1.27)) hide)
     )
@@
   (symbol (lib_id "Werner_custom:TMC0430") (at 92.71 57.15 0) (unit 1)
     (in_bom yes) (on_board yes)
-    (property "Reference" "U24" (id 0) (at 99.06 27.94 0)
+    (property "Reference" "U27" (id 0) (at 99.06 27.94 0)
       (effects (font (size 1.27 1.27)) (justify left))
     )
@@
   (symbol (lib_id "power:VSS") (at 97.79 92.71 0) (unit 1)
     (in_bom yes) (on_board yes)
-    (property "Reference" "#PWR079" (id 0) (at 97.79 96.52 0)
+    (property "Reference" "#PWR081" (id 0) (at 97.79 96.52 0)
       (effects (font (size 1.27 1.27)) hide)
     )
@@
   (symbol (lib_id "Werner_custom:TMC0430") (at 46.99 57.15 0) (unit 1)
     (in_bom yes) (on_board yes)
-    (property "Reference" "U23" (id 0) (at 54.61 27.94 0)
-      (effects (font (size 1.27 1.27)) (justify left))
-    )
+    (property "Reference" "U26" (id 0) (at 54.61 27.94 0)
+      (effects (font (size 1.27 1.27)) (justify left))
+    )
