File: mainboard/ROM-RAM-Sound.kicad_sch (KiCad schematic)
At the start: 13 parts, among them J6 ROM Select, J7 ROM Select, J8 VIDEO OUT, U30 HM62256BLP, U31 HM62256BLP, U32 27C64, U33 27C64, U34 SN76489

Commit message: PCB routed
Parts:
- J6, J7: footprint (none) -> Connector_PinHeader_2.54mm:PinHeader_1x03_P2.54mm_Vertical
- J8: value VIDEO OUT -> AUDIO OUT; footprint (none) -> Connector_PinHeader_2.54mm:PinHeader_1x02_P2.54mm_Vertical
- U29: renamed from U30; footprint Package_DIP:DIP-28_W15.24mm_LongPads -> Package_DIP:DIP-28_W15.24mm_Socket_LongPads
- U30: renamed from U31; footprint Package_DIP:DIP-28_W15.24mm_LongPads -> Package_DIP:DIP-28_W15.24mm_Socket_LongPads
- U31: renamed from U32; footprint Package_DIP:DIP-28_W15.24mm_LongPads -> Package_DIP:DIP-28_W15.24mm_Socket_LongPads
- U32: renamed from U33; footprint Package_DIP:DIP-28_W15.24mm_LongPads -> Package_DIP:DIP-28_W15.24mm_Socket_LongPads
- U33: renamed from U34; footprint Package_DIP:DIP-16_W7.62mm_LongPads -> Package_DIP:DIP-16_W7.62mm_Socket_LongPads
Connections:
- no-connect marks 0 -> 2
Changed lines of the file:
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@@
   (junction (at 127 74.93) (diameter 0) (color 0 0 0 0)
   )
+  (no_connect (at 132.08 66.04))
+  (no_connect (at 132.08 119.38))
   (wire (pts (xy 170.18 139.7) (xy 170.18 143.51))
     (stroke (width 0) (type default) (color 0 0 0 0))
@@
   (symbol (lib_id "TI-Customs:SN76489") (at 236.22 96.52 0) (unit 1)
     (in_bom yes) (on_board yes)
-    (property "Reference" "U34" (id 0) (at 245.11 83.82 0)
+    (property "Reference" "U33" (id 0) (at 245.11 83.82 0)
       (effects (font (size 1.524 1.524)) (justify right))
     )
@@
       (effects (font (size 1.524 1.524)))
     )
-    (property "Footprint" "Package_DIP:DIP-16_W7.62mm_LongPads" (id 2) (at 236.22 96.52 0)
+    (property "Footprint" "Package_DIP:DIP-16_W7.62mm_Socket_LongPads" (id 2) (at 236.22 96.52 0)
       (effects (font (size 1.524 1.524)) hide)
     )
@@
     (property "Reference" "J7" (id 0) (at 120.015 96.52 0))
     (property "Value" "ROM Select" (id 1) (at 120.015 99.06 0))
-    (property "Footprint" "" (id 2) (at 119.38 104.14 0)
+    (property "Footprint" "Connector_PinHeader_2.54mm:PinHeader_1x03_P2.54mm_Vertical" (id 2) (at 119.38 104.14 0)
       (effects (font (size 1.27 1.27)) hide)
     )
@@
   (symbol (lib_id "Memory_EPROM:27C64") (at 149.86 129.54 270) (unit 1)
     (in_bom yes) (on_board yes) (fields_autoplaced)
-    (property "Reference" "U33" (id 0) (at 119.38 122.9612 90))
+    (property "Reference" "U32" (id 0) (at 119.38 122.9612 90))
     (property "Value" "27C64" (id 1) (at 119.38 125.5012 90))
-    (property "Footprint" "Package_DIP:DIP-28_W15.24mm_LongPads" (id 2) (at 149.86 129.54 0)
+    (property "Footprint" "Package_DIP:DIP-28_W15.24mm_Socket_LongPads" (id 2) (at 149.86 129.54 0)
       (effects (font (size 1.27 1.27)) hide)
     )
@@
   (symbol (lib_id "Memory_RAM:HM62256BLP") (at 68.58 69.85 90) (unit 1)
     (in_bom yes) (on_board yes)
-    (property "Reference" "U30" (id 0) (at 96.52 66.2686 90))
+    (property "Reference" "U29" (id 0) (at 96.52 66.2686 90))
     (property "Value" "HM62256BLP" (id 1) (at 96.52 63.5 90))
-    (property "Footprint" "Package_DIP:DIP-28_W15.24mm_LongPads" (id 2) (at 71.12 69.85 0)
+    (property "Footprint" "Package_DIP:DIP-28_W15.24mm_Socket_LongPads" (id 2) (at 71.12 69.85 0)
       (effects (font (size 1.27 1.27)) hide)
     )
@@
       (effects (font (size 1.27 1.27)) (justify right))
     )
-    (property "Value" "VIDEO OUT" (id 1) (at 234.3912 127.5842 0)
+    (property "Value" "AUDIO OUT" (id 1) (at 234.3912 127.5842 0)
       (effects (font (size 1.27 1.27)) (justify right))
     )
-    (property "Footprint" "" (id 2) (at 233.68 128.27 0)
+    (property "Footprint" "Connector_PinHeader_2.54mm:PinHeader_1x02_P2.54mm_Vertical" (id 2) (at 233.68 128.27 0)
       (effects (font (size 1.27 1.27)) hide)
     )
@@
   (symbol (lib_id "Memory_RAM:HM62256BLP") (at 69.85 119.38 90) (mirror x) (unit 1)
     (in_bom yes) (on_board yes) (fields_autoplaced)
-    (property "Reference" "U31" (id 0) (at 97.79 112.8012 90))
+    (property "Reference" "U30" (id 0) (at 97.79 112.8012 90))
     (property "Value" "HM62256BLP" (id 1) (at 97.79 115.3412 90))
-    (property "Footprint" "Package_DIP:DIP-28_W15.24mm_LongPads" (id 2) (at 72.39 119.38 0)
+    (property "Footprint" "Package_DIP:DIP-28_W15.24mm_Socket_LongPads" (id 2) (at 72.39 119.38 0)
       (effects (font (size 1.27 1.27)) hide)
     )
@@
   (symbol (lib_id "Memory_EPROM:27C64") (at 149.86 55.88 270) (mirror x) (unit 1)
     (in_bom yes) (on_board yes) (fields_autoplaced)
-    (property "Reference" "U32" (id 0) (at 119.38 62.4588 90))
+    (property "Reference" "U31" (id 0) (at 119.38 62.4588 90))
     (property "Value" "27C64" (id 1) (at 119.38 59.9188 90))
-    (property "Footprint" "Package_DIP:DIP-28_W15.24mm_LongPads" (id 2) (at 149.86 55.88 0)
+    (property "Footprint" "Package_DIP:DIP-28_W15.24mm_Socket_LongPads" (id 2) (at 149.86 55.88 0)
       (effects (font (size 1.27 1.27)) hide)
     )
@@
     (property "Reference" "J6" (id 0) (at 120.015 88.9 0))
     (property "Value" "ROM Select" (id 1) (at 120.015 86.36 0))
-    (property "Footprint" "" (id 2) (at 119.38 81.28 0)
-      (effects (font (size 1.27 1.27)) hide)
-    )
+    (property "Footprint" "Connector_PinHeader_2.54mm:PinHeader_1x03_P2.54mm_Vertical" (id 2) (at 119.38 81.28 0)
+      (effects (font (size 1.27 1.27)) hide)
+    )

Commit message: unicorn work
Parts:
- C44: renamed from C52; footprint Capacitor_THT:C_Rect_L7.0mm_W2.0mm_P5.00mm -> Capacitor_THT:CP_Radial_D5.0mm_P2.00mm
- renumbered C53 to C45, C54 to C46, R32 to R28, U29 to U25, U30 to U26, U31 to U27, U32 to U28, U33 to U29
Changed lines of the file:
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@@
   (title_block
     (title "TI-99/22")
-    (date "2022-06-23")
-    (rev "0.75")
+    (date "2022-10-11")
+    (rev "0.76")
     (company "Dan Werner - https://github.com/danwerner21/ti99_22")
     (comment 3 "was based on the HackMac KiCAD Design")
@@
   (symbol (lib_id "Console-rescue:GND") (at 120.65 110.49 0) (unit 1)
     (in_bom yes) (on_board yes)
-    (property "Reference" "#PWR0108" (id 0) (at 120.65 116.84 0)
+    (property "Reference" "#PWR090" (id 0) (at 120.65 116.84 0)
       (effects (font (size 1.27 1.27)) hide)
     )
@@
   (symbol (lib_id "Console-rescue:+5V") (at 43.18 69.85 90) (unit 1)
     (in_bom yes) (on_board yes)
-    (property "Reference" "#PWR099" (id 0) (at 46.99 69.85 0)
+    (property "Reference" "#PWR081" (id 0) (at 46.99 69.85 0)
       (effects (font (size 1.27 1.27)) hide)
     )
@@
   (symbol (lib_id "Console-rescue:+5V") (at 44.45 119.38 90) (unit 1)
     (in_bom yes) (on_board yes)
-    (property "Reference" "#PWR0100" (id 0) (at 48.26 119.38 0)
+    (property "Reference" "#PWR082" (id 0) (at 48.26 119.38 0)
       (effects (font (size 1.27 1.27)) hide)
     )
@@
   (symbol (lib_id "Console-rescue:GND") (at 93.98 119.38 90) (unit 1)
     (in_bom yes) (on_board yes)
-    (property "Reference" "#PWR0104" (id 0) (at 100.33 119.38 0)
+    (property "Reference" "#PWR086" (id 0) (at 100.33 119.38 0)
       (effects (font (size 1.27 1.27)) hide)
     )
@@
   (symbol (lib_id "Console-rescue:GND") (at 93.98 69.85 90) (unit 1)
     (in_bom yes) (on_board yes)
-    (property "Reference" "#PWR0103" (id 0) (at 100.33 69.85 0)
+    (property "Reference" "#PWR085" (id 0) (at 100.33 69.85 0)
       (effects (font (size 1.27 1.27)) hide)
     )
@@
   (symbol (lib_id "Console-rescue:+5V") (at 177.8 129.54 270) (unit 1)
     (in_bom yes) (on_board yes)
-    (property "Reference" "#PWR0114" (id 0) (at 173.99 129.54 0)
+    (property "Reference" "#PWR096" (id 0) (at 173.99 129.54 0)
       (effects (font (size 1.27 1.27)) hide)
     )
@@
   (symbol (lib_id "Console-rescue:GND") (at 119.38 129.54 270) (unit 1)
     (in_bom yes) (on_board yes)
-    (property "Reference" "#PWR0106" (id 0) (at 113.03 129.54 0)
+    (property "Reference" "#PWR088" (id 0) (at 113.03 129.54 0)
       (effects (font (size 1.27 1.27)) hide)
     )
@@
   (symbol (lib_id "TI-Customs:SN76489") (at 236.22 96.52 0) (unit 1)
     (in_bom yes) (on_board yes)
-    (property "Reference" "U33" (id 0) (at 245.11 83.82 0)
+    (property "Reference" "U29" (id 0) (at 245.11 83.82 0)
       (effects (font (size 1.524 1.524)) (justify right))
     )
@@
   (symbol (lib_id "Device:CP_Small") (at 195.58 102.87 270) (mirror x) (unit 1)
     (in_bom yes) (on_board yes)
-    (property "Reference" "C52" (id 0) (at 195.58 105.41 90))
+    (property "Reference" "C44" (id 0) (at 195.58 105.41 90))
     (property "Value" "100µF" (id 1) (at 193.04 100.33 90)
       (effects (font (size 1.27 1.27)) (justify left))
     )
-    (property "Footprint" "Capacitor_THT:C_Rect_L7.0mm_W2.0mm_P5.00mm" (id 2) (at 195.58 102.87 0)
+    (property "Footprint" "Capacitor_THT:CP_Radial_D5.0mm_P2.00mm" (id 2) (at 195.58 102.87 0)
       (effects (font (size 1.524 1.524)) hide)
     )
@@
   (symbol (lib_id "TI-Customs:C_Small") (at 201.93 107.95 0) (mirror y) (unit 1)
     (in_bom yes) (on_board yes)
-    (property "Reference" "C53" (id 0) (at 204.47 106.68 0)
+    (property "Reference" "C45" (id 0) (at 204.47 106.68 0)
       (effects (font (size 1.27 1.27)) (justify right))
     )
@@
   (symbol (lib_id "Console-rescue:R_Small") (at 201.93 114.3 0) (mirror y) (unit 1)
     (in_bom yes) (on_board yes)
-    (property "Reference" "R32" (id 0) (at 200.66 113.03 0)
+    (property "Reference" "R28" (id 0) (at 200.66 113.03 0)
       (effects (font (size 1.27 1.27)) (justify left))
     )
@@
   (symbol (lib_id "Console-rescue:GND") (at 201.93 119.38 0) (mirror y) (unit 1)
     (in_bom yes) (on_board yes)
-    (property "Reference" "#PWR0115" (id 0) (at 201.93 125.73 0)
+    (property "Reference" "#PWR097" (id 0) (at 201.93 125.73 0)
       (effects (font (size 1.27 1.27)) hide)
     )
@@
   (symbol (lib_id "TI-Customs:C_Small") (at 240.03 76.2 270) (unit 1)
     (in_bom yes) (on_board yes)
-    (property "Reference" "C54" (id 0) (at 240.03 73.66 90))
+    (property "Reference" "C46" (id 0) (at 240.03 73.66 90))
     (property "Value" "0.1µF" (id 1) (at 240.03 78.74 90))
     (property "Footprint" "Capacitor_THT:C_Rect_L7.0mm_W2.0mm_P5.00mm" (id 2) (at 240.03 76.2 0)
@@
   (symbol (lib_id "Console-rescue:GND") (at 246.38 76.2 0) (unit 1)
     (in_bom yes) (on_board yes)
-    (property "Reference" "#PWR0118" (id 0) (at 246.38 82.55 0)
+    (property "Reference" "#PWR0100" (id 0) (at 246.38 82.55 0)
       (effects (font (size 1.27 1.27)) hide)
     )
@@
   (symbol (lib_id "Console-rescue:+5V") (at 218.44 76.2 0) (unit 1)
     (in_bom yes) (on_board yes)
-    (property "Reference" "#PWR0116" (id 0) (at 218.44 80.01 0)
+    (property "Reference" "#PWR098" (id 0) (at 218.44 80.01 0)
       (effects (font (size 1.27 1.27)) hide)
     )
@@
   (symbol (lib_id "Console-rescue:GND") (at 236.22 107.95 0) (unit 1)
     (in_bom yes) (on_board yes)
-    (property "Reference" "#PWR0117" (id 0) (at 236.22 114.3 0)
+    (property "Reference" "#PWR099" (id 0) (at 236.22 114.3 0)
       (effects (font (size 1.27 1.27)) hide)
     )
@@
   (symbol (lib_id "Console-rescue:+5V") (at 127 101.6 270) (unit 1)
     (in_bom yes) (on_board yes)
-    (property "Reference" "#PWR0110" (id 0) (at 123.19 101.6 0)
+    (property "Reference" "#PWR092" (id 0) (at 123.19 101.6 0)
       (effects (font (size 1.27 1.27)) hide)
     )
@@
   (symbol (lib_id "Console-rescue:+5V") (at 134.62 114.3 0) (unit 1)
     (in_bom yes) (on_board yes)
-    (property "Reference" "#PWR0112" (id 0) (at 134.62 118.11 0)
+    (property "Reference" "#PWR094" (id 0) (at 134.62 118.11 0)
       (effects (font (size 1.27 1.27)) hide)
     )
@@
   (symbol (lib_id "Memory_EPROM:27C64") (at 149.86 129.54 270) (unit 1)
     (in_bom yes) (on_board yes) (fields_autoplaced)
-    (property "Reference" "U32" (id 0) (at 119.38 122.9612 90))
+    (property "Reference" "U28" (id 0) (at 119.38 122.9612 90))
     (property "Value" "27C64" (id 1) (at 119.38 125.5012 90))
     (property "Footprint" "Package_DIP:DIP-28_W15.24mm_Socket_LongPads" (id 2) (at 149.86 129.54 0)
@@
   (symbol (lib_id "Memory_RAM:HM62256BLP") (at 68.58 69.85 90) (unit 1)
     (in_bom yes) (on_board yes)
-    (property "Reference" "U29" (id 0) (at 96.52 66.2686 90))
+    (property "Reference" "U25" (id 0) (at 96.52 66.2686 90))
     (property "Value" "HM62256BLP" (id 1) (at 96.52 63.5 90))
     (property "Footprint" "Package_DIP:DIP-28_W15.24mm_Socket_LongPads" (id 2) (at 71.12 69.85 0)
@@
   (symbol (lib_id "Console-rescue:+5V") (at 127 83.82 270) (mirror x) (unit 1)
     (in_bom yes) (on_board yes)
-    (property "Reference" "#PWR0109" (id 0) (at 123.19 83.82 0)
+    (property "Reference" "#PWR091" (id 0) (at 123.19 83.82 0)
       (effects (font (size 1.27 1.27)) hide)
     )
@@
   (symbol (lib_id "Console-rescue:GND") (at 80.01 46.99 90) (unit 1)
     (in_bom yes) (on_board yes)
-    (property "Reference" "#PWR0101" (id 0) (at 86.36 46.99 0)
+    (property "Reference" "#PWR083" (id 0) (at 86.36 46.99 0)
       (effects (font (size 1.27 1.27)) hide)
     )
@@
   (symbol (lib_id "Console-rescue:GND") (at 80.01 143.51 90) (unit 1)
     (in_bom yes) (on_board yes)
-    (property "Reference" "#PWR0102" (id 0) (at 86.36 143.51 0)
+    (property "Reference" "#PWR084" (id 0) (at 86.36 143.51 0)
       (effects (font (size 1.27 1.27)) hide)
     )
@@
   (symbol (lib_id "Console-rescue:+5V") (at 134.62 71.12 0) (mirror x) (unit 1)
     (in_bom yes) (on_board yes)
-    (property "Reference" "#PWR0111" (id 0) (at 134.62 67.31 0)
+    (property "Reference" "#PWR093" (id 0) (at 134.62 67.31 0)
       (effects (font (size 1.27 1.27)) hide)
     )
@@
   (symbol (lib_id "Memory_RAM:HM62256BLP") (at 69.85 119.38 90) (mirror x) (unit 1)
     (in_bom yes) (on_board yes) (fields_autoplaced)
-    (property "Reference" "U30" (id 0) (at 97.79 112.8012 90))
+    (property "Reference" "U26" (id 0) (at 97.79 112.8012 90))
     (property "Value" "HM62256BLP" (id 1) (at 97.79 115.3412 90))
     (property "Footprint" "Package_DIP:DIP-28_W15.24mm_Socket_LongPads" (id 2) (at 72.39 119.38 0)
@@
   (symbol (lib_id "Memory_EPROM:27C64") (at 149.86 55.88 270) (mirror x) (unit 1)
     (in_bom yes) (on_board yes) (fields_autoplaced)
-    (property "Reference" "U31" (id 0) (at 119.38 62.4588 90))
+    (property "Reference" "U27" (id 0) (at 119.38 62.4588 90))
     (property "Value" "27C64" (id 1) (at 119.38 59.9188 90))
     (property "Footprint" "Package_DIP:DIP-28_W15.24mm_Socket_LongPads" (id 2) (at 149.86 55.88 0)
@@
   (symbol (lib_id "Console-rescue:GND") (at 120.65 74.93 0) (mirror x) (unit 1)
     (in_bom yes) (on_board yes)
-    (property "Reference" "#PWR0107" (id 0) (at 120.65 68.58 0)
+    (property "Reference" "#PWR089" (id 0) (at 120.65 68.58 0)
       (effects (font (size 1.27 1.27)) hide)
     )
@@
   (symbol (lib_id "Console-rescue:GND") (at 119.38 55.88 270) (mirror x) (unit 1)
     (in_bom yes) (on_board yes)
-    (property "Reference" "#PWR0105" (id 0) (at 113.03 55.88 0)
+    (property "Reference" "#PWR087" (id 0) (at 113.03 55.88 0)
       (effects (font (size 1.27 1.27)) hide)
     )
@@
   (symbol (lib_id "Console-rescue:+5V") (at 177.8 55.88 270) (mirror x) (unit 1)
     (in_bom yes) (on_board yes)
-    (property "Reference" "#PWR0113" (id 0) (at 173.99 55.88 0)
-      (effects (font (size 1.27 1.27)) hide)
-    )
+    (property "Reference" "#PWR095" (id 0) (at 173.99 55.88 0)
+      (effects (font (size 1.27 1.27)) hide)
+    )

Commit message: unicorn work
Parts:
- renumbered C44 to C52, C45 to C53, C46 to C54
Changed lines of the file:
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@@
   (symbol (lib_id "Console-rescue:GND") (at 120.65 110.49 0) (unit 1)
     (in_bom yes) (on_board yes)
-    (property "Reference" "#PWR090" (id 0) (at 120.65 116.84 0)
+    (property "Reference" "#PWR091" (id 0) (at 120.65 116.84 0)
       (effects (font (size 1.27 1.27)) hide)
     )
@@
   (symbol (lib_id "Console-rescue:+5V") (at 43.18 69.85 90) (unit 1)
     (in_bom yes) (on_board yes)
-    (property "Reference" "#PWR081" (id 0) (at 46.99 69.85 0)
+    (property "Reference" "#PWR082" (id 0) (at 46.99 69.85 0)
       (effects (font (size 1.27 1.27)) hide)
     )
@@
   (symbol (lib_id "Console-rescue:+5V") (at 44.45 119.38 90) (unit 1)
     (in_bom yes) (on_board yes)
-    (property "Reference" "#PWR082" (id 0) (at 48.26 119.38 0)
+    (property "Reference" "#PWR083" (id 0) (at 48.26 119.38 0)
       (effects (font (size 1.27 1.27)) hide)
     )
@@
   (symbol (lib_id "Console-rescue:GND") (at 93.98 119.38 90) (unit 1)
     (in_bom yes) (on_board yes)
-    (property "Reference" "#PWR086" (id 0) (at 100.33 119.38 0)
+    (property "Reference" "#PWR087" (id 0) (at 100.33 119.38 0)
       (effects (font (size 1.27 1.27)) hide)
     )
@@
   (symbol (lib_id "Console-rescue:GND") (at 93.98 69.85 90) (unit 1)
     (in_bom yes) (on_board yes)
-    (property "Reference" "#PWR085" (id 0) (at 100.33 69.85 0)
+    (property "Reference" "#PWR086" (id 0) (at 100.33 69.85 0)
       (effects (font (size 1.27 1.27)) hide)
     )
@@
   (symbol (lib_id "Console-rescue:+5V") (at 177.8 129.54 270) (unit 1)
     (in_bom yes) (on_board yes)
-    (property "Reference" "#PWR096" (id 0) (at 173.99 129.54 0)
+    (property "Reference" "#PWR097" (id 0) (at 173.99 129.54 0)
       (effects (font (size 1.27 1.27)) hide)
     )
@@
   (symbol (lib_id "Console-rescue:GND") (at 119.38 129.54 270) (unit 1)
     (in_bom yes) (on_board yes)
-    (property "Reference" "#PWR088" (id 0) (at 113.03 129.54 0)
+    (property "Reference" "#PWR089" (id 0) (at 113.03 129.54 0)
       (effects (font (size 1.27 1.27)) hide)
     )
@@
   (symbol (lib_id "Device:CP_Small") (at 195.58 102.87 270) (mirror x) (unit 1)
     (in_bom yes) (on_board yes)
-    (property "Reference" "C44" (id 0) (at 195.58 105.41 90))
+    (property "Reference" "C52" (id 0) (at 195.58 105.41 90))
     (property "Value" "100µF" (id 1) (at 193.04 100.33 90)
       (effects (font (size 1.27 1.27)) (justify left))
@@
   (symbol (lib_id "TI-Customs:C_Small") (at 201.93 107.95 0) (mirror y) (unit 1)
     (in_bom yes) (on_board yes)
-    (property "Reference" "C45" (id 0) (at 204.47 106.68 0)
+    (property "Reference" "C53" (id 0) (at 204.47 106.68 0)
       (effects (font (size 1.27 1.27)) (justify right))
     )
@@
   (symbol (lib_id "Console-rescue:GND") (at 201.93 119.38 0) (mirror y) (unit 1)
     (in_bom yes) (on_board yes)
-    (property "Reference" "#PWR097" (id 0) (at 201.93 125.73 0)
+    (property "Reference" "#PWR098" (id 0) (at 201.93 125.73 0)
       (effects (font (size 1.27 1.27)) hide)
     )
@@
   (symbol (lib_id "TI-Customs:C_Small") (at 240.03 76.2 270) (unit 1)
     (in_bom yes) (on_board yes)
-    (property "Reference" "C46" (id 0) (at 240.03 73.66 90))
+    (property "Reference" "C54" (id 0) (at 240.03 73.66 90))
     (property "Value" "0.1µF" (id 1) (at 240.03 78.74 90))
     (property "Footprint" "Capacitor_THT:C_Rect_L7.0mm_W2.0mm_P5.00mm" (id 2) (at 240.03 76.2 0)
@@
   (symbol (lib_id "Console-rescue:GND") (at 246.38 76.2 0) (unit 1)
     (in_bom yes) (on_board yes)
-    (property "Reference" "#PWR0100" (id 0) (at 246.38 82.55 0)
+    (property "Reference" "#PWR0101" (id 0) (at 246.38 82.55 0)
       (effects (font (size 1.27 1.27)) hide)
     )
@@
   (symbol (lib_id "Console-rescue:+5V") (at 218.44 76.2 0) (unit 1)
     (in_bom yes) (on_board yes)
-    (property "Reference" "#PWR098" (id 0) (at 218.44 80.01 0)
+    (property "Reference" "#PWR099" (id 0) (at 218.44 80.01 0)
       (effects (font (size 1.27 1.27)) hide)
     )
@@
   (symbol (lib_id "Console-rescue:GND") (at 236.22 107.95 0) (unit 1)
     (in_bom yes) (on_board yes)
-    (property "Reference" "#PWR099" (id 0) (at 236.22 114.3 0)
+    (property "Reference" "#PWR0100" (id 0) (at 236.22 114.3 0)
       (effects (font (size 1.27 1.27)) hide)
     )
@@
   (symbol (lib_id "Console-rescue:+5V") (at 127 101.6 270) (unit 1)
     (in_bom yes) (on_board yes)
-    (property "Reference" "#PWR092" (id 0) (at 123.19 101.6 0)
+    (property "Reference" "#PWR093" (id 0) (at 123.19 101.6 0)
       (effects (font (size 1.27 1.27)) hide)
     )
@@
   (symbol (lib_id "Console-rescue:+5V") (at 134.62 114.3 0) (unit 1)
     (in_bom yes) (on_board yes)
-    (property "Reference" "#PWR094" (id 0) (at 134.62 118.11 0)
+    (property "Reference" "#PWR095" (id 0) (at 134.62 118.11 0)
       (effects (font (size 1.27 1.27)) hide)
     )
@@
   (symbol (lib_id "Console-rescue:+5V") (at 127 83.82 270) (mirror x) (unit 1)
     (in_bom yes) (on_board yes)
-    (property "Reference" "#PWR091" (id 0) (at 123.19 83.82 0)
+    (property "Reference" "#PWR092" (id 0) (at 123.19 83.82 0)
       (effects (font (size 1.27 1.27)) hide)
     )
@@
   (symbol (lib_id "Console-rescue:GND") (at 80.01 46.99 90) (unit 1)
     (in_bom yes) (on_board yes)
-    (property "Reference" "#PWR083" (id 0) (at 86.36 46.99 0)
+    (property "Reference" "#PWR084" (id 0) (at 86.36 46.99 0)
       (effects (font (size 1.27 1.27)) hide)
     )
@@
   (symbol (lib_id "Console-rescue:GND") (at 80.01 143.51 90) (unit 1)
     (in_bom yes) (on_board yes)
-    (property "Reference" "#PWR084" (id 0) (at 86.36 143.51 0)
+    (property "Reference" "#PWR085" (id 0) (at 86.36 143.51 0)
       (effects (font (size 1.27 1.27)) hide)
     )
@@
   (symbol (lib_id "Console-rescue:+5V") (at 134.62 71.12 0) (mirror x) (unit 1)
     (in_bom yes) (on_board yes)
-    (property "Reference" "#PWR093" (id 0) (at 134.62 67.31 0)
+    (property "Reference" "#PWR094" (id 0) (at 134.62 67.31 0)
       (effects (font (size 1.27 1.27)) hide)
     )
@@
   (symbol (lib_id "Console-rescue:GND") (at 120.65 74.93 0) (mirror x) (unit 1)
     (in_bom yes) (on_board yes)
-    (property "Reference" "#PWR089" (id 0) (at 120.65 68.58 0)
+    (property "Reference" "#PWR090" (id 0) (at 120.65 68.58 0)
       (effects (font (size 1.27 1.27)) hide)
     )
@@
   (symbol (lib_id "Console-rescue:GND") (at 119.38 55.88 270) (mirror x) (unit 1)
     (in_bom yes) (on_board yes)
-    (property "Reference" "#PWR087" (id 0) (at 113.03 55.88 0)
+    (property "Reference" "#PWR088" (id 0) (at 113.03 55.88 0)
       (effects (font (size 1.27 1.27)) hide)
     )
@@
   (symbol (lib_id "Console-rescue:+5V") (at 177.8 55.88 270) (mirror x) (unit 1)
     (in_bom yes) (on_board yes)
-    (property "Reference" "#PWR095" (id 0) (at 173.99 55.88 0)
-      (effects (font (size 1.27 1.27)) hide)
-    )
+    (property "Reference" "#PWR096" (id 0) (at 173.99 55.88 0)
+      (effects (font (size 1.27 1.27)) hide)
+    )
