File: mainboard/ROM-RAM-Sound.kicad_sch (KiCad schematic)
At the start: 13 parts, among them J6 ROM Select, J7 ROM Select, J8 AUDIO OUT, U25 HM62256BLP, U26 HM62256BLP, U27 27C64, U28 27C64, U29 SN76489

Commit message: Shrink PCB
Parts:
- renumbered J6 to J5, J7 to J6, J8 to J7
Changed lines of the file:
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@@
   (symbol (lib_id "Connector:Conn_01x03_Male") (at 119.38 104.14 0) (unit 1)
     (in_bom yes) (on_board yes) (fields_autoplaced)
-    (property "Reference" "J7" (id 0) (at 120.015 96.52 0))
+    (property "Reference" "J6" (id 0) (at 120.015 96.52 0))
     (property "Value" "ROM Select" (id 1) (at 120.015 99.06 0))
     (property "Footprint" "Connector_PinHeader_2.54mm:PinHeader_1x03_P2.54mm_Vertical" (id 2) (at 119.38 104.14 0)
@@
   (symbol (lib_id "Connector:Conn_01x02_Male") (at 233.68 128.27 180) (unit 1)
     (in_bom yes) (on_board yes)
-    (property "Reference" "J8" (id 0) (at 234.3912 125.2728 0)
+    (property "Reference" "J7" (id 0) (at 234.3912 125.2728 0)
       (effects (font (size 1.27 1.27)) (justify right))
     )
@@
   (symbol (lib_id "Connector:Conn_01x03_Male") (at 119.38 81.28 0) (mirror x) (unit 1)
     (in_bom yes) (on_board yes) (fields_autoplaced)
-    (property "Reference" "J6" (id 0) (at 120.015 88.9 0))
+    (property "Reference" "J5" (id 0) (at 120.015 88.9 0))
     (property "Value" "ROM Select" (id 1) (at 120.015 86.36 0))
     (property "Footprint" "Connector_PinHeader_2.54mm:PinHeader_1x03_P2.54mm_Vertical" (id 2) (at 119.38 81.28 0)

Commit message: hardware updates
Parts:
- renumbered L8 to L7, R28 to R27
Changed lines of the file:
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@@
   (symbol (lib_id "Console-rescue:R_Small") (at 201.93 114.3 0) (mirror y) (unit 1)
     (in_bom yes) (on_board yes)
-    (property "Reference" "R28" (id 0) (at 200.66 113.03 0)
+    (property "Reference" "R27" (id 0) (at 200.66 113.03 0)
       (effects (font (size 1.27 1.27)) (justify left))
     )
@@
   (symbol (lib_id "Console-rescue:INDUCTOR_SMALL") (at 228.6 76.2 0) (unit 1)
     (in_bom yes) (on_board yes)
-    (property "Reference" "L8" (id 0) (at 228.6 73.66 0))
+    (property "Reference" "L7" (id 0) (at 228.6 73.66 0))
     (property "Value" "6.8µH" (id 1) (at 228.6 77.47 0))
     (property "Footprint" "Resistor_THT:R_Axial_DIN0207_L6.3mm_D2.5mm_P7.62mm_Horizontal" (id 2) (at 228.6 76.2 0)

Commit message: PCB cleanup
Parts:
- C52: symbol Device:CP_Small -> Device:C_Polarized_Small
- C53, C54: symbol TI-Customs:C_Small -> Device:C
- L7: symbol Console-rescue:INDUCTOR_SMALL -> Device:L
- R27: symbol Console-rescue:R_Small -> Device:R_Small
- U30: renamed from U29; symbol TI-Customs:SN76489 -> Werner_custom:SN76489
- renumbered U25 to U26, U26 to U27, U27 to U28, U28 to U29
Other:
- moved on the sheet: C54, L7

Commit message: PCB rework
Parts:
- removed L7: 6.8µH, Resistor_THT:R_Axial_DIN0207_L6.3mm_D2.5mm_P7.62mm_Horizontal, symbol Device:L
- added J7: Sound Clock Select, Connector_PinHeader_2.54mm:PinHeader_1x03_P2.54mm_Vertical, symbol Connector:Conn_01x03_Male
- renumbered C52 to C53, C53 to C54, C54 to C55, J7 to J8, U26 to U29, U27 to U30, U28 to U31, U29 to U32, U30 to U33
Connections:
- net +5V: now also C55.2, U33.16 (VCC)
- net GRMCLK: now also J7.3 (Pin_3); no longer U33.14 (CLK)
- new net CPUCLK: J7.1 (Pin_1)
- new net SOUNDCLK: J7.2 (Pin_2), U33.14 (CLK)
