File: mainboard/Video.kicad_sch (KiCad schematic)
At the start: 27 parts, among them J9 VIDEO OUT, Q2 2N3904, U21 74LS04, U35 TMS9918, U36 74LS574, U37 74LS574, U38 HM62256BLP, U39 74LS574, U9 74LS32, Y2 10.7MHz

Commit message: PCB routed
Parts:
- C58, C59, C60: footprint Capacitor_THT:C_Rect_L7.0mm_W2.0mm_P5.00mm -> Capacitor_THT:CP_Radial_D7.5mm_P2.50mm
- J9: footprint homecomputer2:CUI_RCJ-041 -> Connector_PinHeader_2.54mm:PinHeader_1x02_P2.54mm_Vertical
- L12: footprint Resistor_THT:R_Axial_DIN0207_L6.3mm_D2.5mm_P15.24mm_Horizontal -> Resistor_THT:R_Axial_DIN0207_L6.3mm_D2.5mm_P7.62mm_Horizontal
- L9: footprint (none) -> Resistor_THT:R_Axial_DIN0207_L6.3mm_D2.5mm_P7.62mm_Horizontal
- U21: footprint Package_DIP:DIP-14_W7.62mm_LongPads -> Package_DIP:DIP-14_W7.62mm_Socket_LongPads
- U34: renamed from U35; footprint Package_DIP:DIP-40_W25.4mm_LongPads -> Package_DIP:DIP-40_W15.24mm_Socket_LongPads
- U35: renamed from U36; footprint Package_DIP:DIP-20_W7.62mm_LongPads -> Package_DIP:DIP-20_W7.62mm_Socket_LongPads
- U36: renamed from U37; footprint Package_DIP:DIP-20_W7.62mm_LongPads -> Package_DIP:DIP-20_W7.62mm_Socket_LongPads
- U37: renamed from U38; footprint Package_DIP:DIP-28_W15.24mm_LongPads -> Package_DIP:DIP-28_W15.24mm_Socket_LongPads
- U38: renamed from U39; footprint Package_DIP:DIP-20_W7.62mm_LongPads -> Package_DIP:DIP-20_W7.62mm_Socket_LongPads
- U9: footprint Package_DIP:DIP-16_W7.62mm_LongPads -> Package_DIP:DIP-14_W7.62mm_Socket_LongPads
- Y2: footprint (none) -> Crystal:Crystal_HC49-U_Vertical
Changed lines of the file:
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@@
-    (stroke (width 0) (type default) (color 0 0 0 0))
-  )
-  (wire (pts (xy 58.42 113.03) (xy 58.42 109.22))
     (stroke (width 0) (type default) (color 0 0 0 0))
   )
@@
       (effects (font (size 1.524 1.524)))
     )
-    (property "Footprint" "Package_DIP:DIP-16_W7.62mm_LongPads" (id 2) (at 43.18 44.45 0)
+    (property "Footprint" "Package_DIP:DIP-14_W7.62mm_Socket_LongPads" (id 2) (at 43.18 44.45 0)
       (effects (font (size 1.524 1.524)) hide)
     )
@@
       (effects (font (size 0.762 0.762)))
     )
-    (property "Footprint" "" (id 2) (at 55.88 96.52 0)
+    (property "Footprint" "Crystal:Crystal_HC49-U_Vertical" (id 2) (at 55.88 96.52 0)
       (effects (font (size 1.524 1.524)) hide)
     )
@@
       (effects (font (size 0.762 0.762)))
     )
-    (property "Footprint" "" (id 2) (at 43.18 96.52 0)
+    (property "Footprint" "Resistor_THT:R_Axial_DIN0207_L6.3mm_D2.5mm_P7.62mm_Horizontal" (id 2) (at 43.18 96.52 0)
       (effects (font (size 1.524 1.524)) hide)
     )
@@
       (effects (font (size 1.27 1.27)) (justify right))
     )
-    (property "Footprint" "Capacitor_THT:C_Rect_L7.0mm_W2.0mm_P5.00mm" (id 2) (at 99.06 33.02 0)
+    (property "Footprint" "Capacitor_THT:CP_Radial_D7.5mm_P2.50mm" (id 2) (at 99.06 33.02 0)
       (effects (font (size 1.524 1.524)) hide)
     )
@@
     (property "Reference" "L12" (id 0) (at 107.95 39.37 0))
     (property "Value" "6.8µH" (id 1) (at 107.95 35.56 0))
-    (property "Footprint" "Resistor_THT:R_Axial_DIN0207_L6.3mm_D2.5mm_P15.24mm_Horizontal" (id 2) (at 107.95 36.83 0)
+    (property "Footprint" "Resistor_THT:R_Axial_DIN0207_L6.3mm_D2.5mm_P7.62mm_Horizontal" (id 2) (at 107.95 36.83 0)
       (effects (font (size 1.524 1.524)) hide)
     )
@@
     (property "Reference" "U21" (id 0) (at 265.43 149.86 0))
     (property "Value" "74LS04" (id 1) (at 265.43 152.4 0))
-    (property "Footprint" "Package_DIP:DIP-14_W7.62mm_LongPads" (id 2) (at 265.43 158.75 0)
+    (property "Footprint" "Package_DIP:DIP-14_W7.62mm_Socket_LongPads" (id 2) (at 265.43 158.75 0)
       (effects (font (size 1.27 1.27)) hide)
     )
@@
     (property "Reference" "U21" (id 0) (at 229.87 149.86 0))
     (property "Value" "74LS04" (id 1) (at 229.87 152.4 0))
-    (property "Footprint" "Package_DIP:DIP-14_W7.62mm_LongPads" (id 2) (at 229.87 158.75 0)
+    (property "Footprint" "Package_DIP:DIP-14_W7.62mm_Socket_LongPads" (id 2) (at 229.87 158.75 0)
       (effects (font (size 1.27 1.27)) hide)
     )
@@
   (symbol (lib_id "Memory_RAM:HM62256BLP") (at 242.57 45.72 0) (unit 1)
     (in_bom yes) (on_board yes)
-    (property "Reference" "U38" (id 0) (at 246.1514 73.66 90))
+    (property "Reference" "U37" (id 0) (at 246.1514 73.66 90))
     (property "Value" "HM62256BLP" (id 1) (at 248.92 73.66 90))
-    (property "Footprint" "Package_DIP:DIP-28_W15.24mm_LongPads" (id 2) (at 242.57 48.26 0)
+    (property "Footprint" "Package_DIP:DIP-28_W15.24mm_Socket_LongPads" (id 2) (at 242.57 48.26 0)
       (effects (font (size 1.27 1.27)) hide)
     )
@@
   (symbol (lib_id "TI:TMS9918") (at 99.06 48.26 0) (unit 1)
     (in_bom yes) (on_board yes) (fields_autoplaced)
-    (property "Reference" "U35" (id 0) (at 101.0794 43.18 0)
+    (property "Reference" "U34" (id 0) (at 101.0794 43.18 0)
       (effects (font (size 1.27 1.27)) (justify left))
     )
@@
       (effects (font (size 1.27 1.27)) (justify left))
     )
-    (property "Footprint" "Package_DIP:DIP-40_W25.4mm_LongPads" (id 2) (at 99.06 48.26 0)
+    (property "Footprint" "Package_DIP:DIP-40_W15.24mm_Socket_LongPads" (id 2) (at 99.06 48.26 0)
       (effects (font (size 1.27 1.27)) hide)
     )
@@
       (effects (font (size 1.27 1.27)) (justify right))
     )
-    (property "Footprint" "homecomputer2:CUI_RCJ-041" (id 2) (at 137.16 175.26 0)
+    (property "Footprint" "Connector_PinHeader_2.54mm:PinHeader_1x02_P2.54mm_Vertical" (id 2) (at 137.16 175.26 0)
       (effects (font (size 1.27 1.27)) hide)
     )
@@
       (effects (font (size 1.27 1.27)) (justify left))
     )
-    (property "Footprint" "Capacitor_THT:C_Rect_L7.0mm_W2.0mm_P5.00mm" (id 2) (at 109.22 172.72 0)
+    (property "Footprint" "Capacitor_THT:CP_Radial_D7.5mm_P2.50mm" (id 2) (at 109.22 172.72 0)
       (effects (font (size 1.524 1.524)) hide)
     )
@@
     (property "Reference" "U21" (id 0) (at 247.65 149.86 0))
     (property "Value" "74LS04" (id 1) (at 247.65 152.4 0))
-    (property "Footprint" "Package_DIP:DIP-14_W7.62mm_LongPads" (id 2) (at 247.65 158.75 0)
+    (property "Footprint" "Package_DIP:DIP-14_W7.62mm_Socket_LongPads" (id 2) (at 247.65 158.75 0)
       (effects (font (size 1.27 1.27)) hide)
     )
@@
   (symbol (lib_id "74xx:74LS574") (at 243.84 110.49 0) (unit 1)
     (in_bom yes) (on_board yes) (fields_autoplaced)
-    (property "Reference" "U39" (id 0) (at 245.8594 91.44 0)
+    (property "Reference" "U38" (id 0) (at 245.8594 91.44 0)
       (effects (font (size 1.27 1.27)) (justify left))
     )
@@
       (effects (font (size 1.27 1.27)) (justify left))
     )
-    (property "Footprint" "Package_DIP:DIP-20_W7.62mm_LongPads" (id 2) (at 243.84 110.49 0)
+    (property "Footprint" "Package_DIP:DIP-20_W7.62mm_Socket_LongPads" (id 2) (at 243.84 110.49 0)
       (effects (font (size 1.27 1.27)) hide)
     )
@@
     (property "Reference" "U21" (id 0) (at 198.12 148.59 0))
     (property "Value" "74LS04" (id 1) (at 198.12 146.05 0))
-    (property "Footprint" "Package_DIP:DIP-14_W7.62mm_LongPads" (id 2) (at 199.39 139.7 0)
+    (property "Footprint" "Package_DIP:DIP-14_W7.62mm_Socket_LongPads" (id 2) (at 199.39 139.7 0)
       (effects (font (size 1.27 1.27)) hide)
     )
@@
   (symbol (lib_id "74xx:74LS574") (at 173.99 40.64 0) (unit 1)
     (in_bom yes) (on_board yes) (fields_autoplaced)
-    (property "Reference" "U36" (id 0) (at 176.0094 21.59 0)
+    (property "Reference" "U35" (id 0) (at 176.0094 21.59 0)
       (effects (font (size 1.27 1.27)) (justify left))
     )
@@
       (effects (font (size 1.27 1.27)) (justify left))
     )
-    (property "Footprint" "Package_DIP:DIP-20_W7.62mm_LongPads" (id 2) (at 173.99 40.64 0)
+    (property "Footprint" "Package_DIP:DIP-20_W7.62mm_Socket_LongPads" (id 2) (at 173.99 40.64 0)
       (effects (font (size 1.27 1.27)) hide)
     )
@@
       (effects (font (size 1.27 1.27)) (justify left))
     )
-    (property "Footprint" "Capacitor_THT:C_Rect_L7.0mm_W2.0mm_P5.00mm" (id 2) (at 97.79 160.02 0)
+    (property "Footprint" "Capacitor_THT:CP_Radial_D7.5mm_P2.50mm" (id 2) (at 97.79 160.02 0)
       (effects (font (size 1.524 1.524)) hide)
     )
@@
   (symbol (lib_id "74xx:74LS574") (at 173.99 90.17 0) (unit 1)
     (in_bom yes) (on_board yes) (fields_autoplaced)
-    (property "Reference" "U37" (id 0) (at 176.0094 71.12 0)
+    (property "Reference" "U36" (id 0) (at 176.0094 71.12 0)
       (effects (font (size 1.27 1.27)) (justify left))
     )
@@
       (effects (font (size 1.27 1.27)) (justify left))
     )
-    (property "Footprint" "Package_DIP:DIP-20_W7.62mm_LongPads" (id 2) (at 173.99 90.17 0)
+    (property "Footprint" "Package_DIP:DIP-20_W7.62mm_Socket_LongPads" (id 2) (at 173.99 90.17 0)
       (effects (font (size 1.27 1.27)) hide)
     )
@@
     (property "Reference" "U21" (id 0) (at 199.39 121.92 0))
     (property "Value" "74LS04" (id 1) (at 199.39 124.46 0))
-    (property "Footprint" "Package_DIP:DIP-14_W7.62mm_LongPads" (id 2) (at 199.39 130.81 0)
-      (effects (font (size 1.27 1.27)) hide)
-    )
+    (property "Footprint" "Package_DIP:DIP-14_W7.62mm_Socket_LongPads" (id 2) (at 199.39 130.81 0)
+      (effects (font (size 1.27 1.27)) hide)
+    )

Commit message: unicorn work
Parts:
- renumbered C55 to C47, C56 to C48, C57 to C49, C58 to C50, C59 to C51, C60 to C52, C61 to C53, R33 to R29, R34 to R30, R35 to R31, R36 to R32, R37 to R33, R38 to R34, U34 to U30, U35 to U31, U36 to U32, U37 to U33, U38 to U34
Connections:
- net VRAM_BANK is gone; now on net GND: U33.1 (A14)

Commit message: unicorn work
Parts:
- renumbered C47 to C55, C48 to C56, C49 to C57, C50 to C58, C51 to C59, C52 to C60, C53 to C61
Changed lines of the file:
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@@
   (symbol (lib_id "TI-Customs:C_Small") (at 33.02 102.87 0) (unit 1)
     (in_bom yes) (on_board yes)
-    (property "Reference" "C47" (id 0) (at 25.4 101.6 0)
+    (property "Reference" "C55" (id 0) (at 25.4 101.6 0)
       (effects (font (size 1.27 1.27)) (justify left))
     )
@@
   (symbol (lib_id "TI-Customs:C_Small") (at 63.5 102.87 0) (unit 1)
     (in_bom yes) (on_board yes)
-    (property "Reference" "C48" (id 0) (at 69.85 100.33 0)
+    (property "Reference" "C56" (id 0) (at 69.85 100.33 0)
       (effects (font (size 1.27 1.27)) (justify right))
     )
@@
   (symbol (lib_id "Console-rescue:GND") (at 63.5 105.41 0) (unit 1)
     (in_bom yes) (on_board yes)
-    (property "Reference" "#PWR0103" (id 0) (at 63.5 111.76 0)
+    (property "Reference" "#PWR0104" (id 0) (at 63.5 111.76 0)
       (effects (font (size 1.27 1.27)) hide)
     )
@@
   (symbol (lib_id "Console-rescue:GND") (at 33.02 105.41 0) (unit 1)
     (in_bom yes) (on_board yes)
-    (property "Reference" "#PWR0101" (id 0) (at 33.02 111.76 0)
+    (property "Reference" "#PWR0102" (id 0) (at 33.02 111.76 0)
       (effects (font (size 1.27 1.27)) hide)
     )
@@
   (symbol (lib_id "Device:CP") (at 99.06 33.02 0) (mirror x) (unit 1)
     (in_bom yes) (on_board yes)
-    (property "Reference" "C51" (id 0) (at 106.68 30.48 0)
+    (property "Reference" "C59" (id 0) (at 106.68 30.48 0)
       (effects (font (size 1.27 1.27)) (justify right))
     )
@@
   (symbol (lib_id "TI-Customs:C_Small") (at 92.71 33.02 180) (unit 1)
     (in_bom yes) (on_board yes)
-    (property "Reference" "C49" (id 0) (at 92.456 34.798 0)
+    (property "Reference" "C57" (id 0) (at 92.456 34.798 0)
       (effects (font (size 1.27 1.27)) (justify left))
     )
@@
   (symbol (lib_id "power:+5V") (at 114.3 36.83 0) (unit 1)
     (in_bom yes) (on_board yes) (fields_autoplaced)
-    (property "Reference" "#PWR0109" (id 0) (at 114.3 40.64 0)
+    (property "Reference" "#PWR0110" (id 0) (at 114.3 40.64 0)
       (effects (font (size 1.27 1.27)) hide)
     )
@@
   (symbol (lib_id "Console-rescue:GND") (at 243.84 133.35 0) (unit 1)
     (in_bom yes) (on_board yes)
-    (property "Reference" "#PWR0120" (id 0) (at 243.84 139.7 0)
+    (property "Reference" "#PWR0121" (id 0) (at 243.84 139.7 0)
       (effects (font (size 1.27 1.27)) hide)
     )
@@
   (symbol (lib_id "Console-rescue:GND") (at 242.57 68.58 0) (unit 1)
     (in_bom yes) (on_board yes)
-    (property "Reference" "#PWR0118" (id 0) (at 242.57 74.93 0)
+    (property "Reference" "#PWR0119" (id 0) (at 242.57 74.93 0)
       (effects (font (size 1.27 1.27)) hide)
     )
@@
   (symbol (lib_id "Console-rescue:GND") (at 62.23 172.72 0) (unit 1)
     (in_bom yes) (on_board yes)
-    (property "Reference" "#PWR0102" (id 0) (at 62.23 179.07 0)
+    (property "Reference" "#PWR0103" (id 0) (at 62.23 179.07 0)
       (effects (font (size 1.27 1.27)) hide)
     )
@@
   (symbol (lib_id "Console-rescue:GND") (at 99.06 111.76 0) (unit 1)
     (in_bom yes) (on_board yes)
-    (property "Reference" "#PWR0107" (id 0) (at 99.06 118.11 0)
+    (property "Reference" "#PWR0108" (id 0) (at 99.06 118.11 0)
       (effects (font (size 1.27 1.27)) hide)
     )
@@
   (symbol (lib_id "Console-rescue:GND") (at 173.99 114.3 0) (unit 1)
     (in_bom yes) (on_board yes)
-    (property "Reference" "#PWR0116" (id 0) (at 173.99 120.65 0)
+    (property "Reference" "#PWR0117" (id 0) (at 173.99 120.65 0)
       (effects (font (size 1.27 1.27)) hide)
     )
@@
   (symbol (lib_id "Console-rescue:GND") (at 85.09 177.8 0) (unit 1)
     (in_bom yes) (on_board yes)
-    (property "Reference" "#PWR0104" (id 0) (at 85.09 184.15 0)
+    (property "Reference" "#PWR0105" (id 0) (at 85.09 184.15 0)
       (effects (font (size 1.27 1.27)) hide)
     )
@@
   (symbol (lib_id "power:+5V") (at 243.84 88.9 0) (unit 1)
     (in_bom yes) (on_board yes) (fields_autoplaced)
-    (property "Reference" "#PWR0119" (id 0) (at 243.84 92.71 0)
+    (property "Reference" "#PWR0120" (id 0) (at 243.84 92.71 0)
       (effects (font (size 1.27 1.27)) hide)
     )
@@
   (symbol (lib_id "Console-rescue:GND") (at 99.06 29.21 180) (unit 1)
     (in_bom yes) (on_board yes)
-    (property "Reference" "#PWR0106" (id 0) (at 99.06 22.86 0)
+    (property "Reference" "#PWR0107" (id 0) (at 99.06 22.86 0)
       (effects (font (size 1.27 1.27)) hide)
     )
@@
   (symbol (lib_id "HC3-rescue:C") (at 110.49 160.02 0) (unit 1)
     (in_bom yes) (on_board yes)
-    (property "Reference" "C53" (id 0) (at 111.76 157.48 0)
+    (property "Reference" "C61" (id 0) (at 111.76 157.48 0)
       (effects (font (size 1.27 1.27)) (justify left))
     )
@@
   (symbol (lib_id "power:+5V") (at 97.79 139.7 0) (unit 1)
     (in_bom yes) (on_board yes) (fields_autoplaced)
-    (property "Reference" "#PWR0105" (id 0) (at 97.79 143.51 0)
+    (property "Reference" "#PWR0106" (id 0) (at 97.79 143.51 0)
       (effects (font (size 1.27 1.27)) hide)
     )
@@
   (symbol (lib_id "Console-rescue:GND") (at 148.59 53.34 0) (unit 1)
     (in_bom yes) (on_board yes)
-    (property "Reference" "#PWR0111" (id 0) (at 148.59 59.69 0)
+    (property "Reference" "#PWR0112" (id 0) (at 148.59 59.69 0)
       (effects (font (size 1.27 1.27)) hide)
     )
@@
   (symbol (lib_id "power:+5V") (at 173.99 68.58 0) (unit 1)
     (in_bom yes) (on_board yes)
-    (property "Reference" "#PWR0115" (id 0) (at 173.99 72.39 0)
+    (property "Reference" "#PWR0116" (id 0) (at 173.99 72.39 0)
       (effects (font (size 1.27 1.27)) hide)
     )
@@
   (symbol (lib_id "Console-rescue:GND") (at 128.27 184.15 0) (unit 1)
     (in_bom yes) (on_board yes)
-    (property "Reference" "#PWR0110" (id 0) (at 128.27 190.5 0)
+    (property "Reference" "#PWR0111" (id 0) (at 128.27 190.5 0)
       (effects (font (size 1.27 1.27)) hide)
     )
@@
   (symbol (lib_id "Console-rescue:GND") (at 110.49 165.1 0) (unit 1)
     (in_bom yes) (on_board yes)
-    (property "Reference" "#PWR0108" (id 0) (at 110.49 171.45 0)
+    (property "Reference" "#PWR0109" (id 0) (at 110.49 171.45 0)
       (effects (font (size 1.27 1.27)) hide)
     )
@@
   (symbol (lib_id "Console-rescue:GND") (at 148.59 102.87 0) (unit 1)
     (in_bom yes) (on_board yes)
-    (property "Reference" "#PWR0112" (id 0) (at 148.59 109.22 0)
+    (property "Reference" "#PWR0113" (id 0) (at 148.59 109.22 0)
       (effects (font (size 1.27 1.27)) hide)
     )
@@
   (symbol (lib_id "HC3-rescue:CP") (at 109.22 172.72 90) (mirror x) (unit 1)
     (in_bom yes) (on_board yes)
-    (property "Reference" "C52" (id 0) (at 106.68 173.99 0)
+    (property "Reference" "C60" (id 0) (at 106.68 173.99 0)
       (effects (font (size 1.27 1.27)) (justify left))
     )
@@
   (symbol (lib_id "Console-rescue:GND") (at 173.99 62.23 0) (unit 1)
     (in_bom yes) (on_board yes)
-    (property "Reference" "#PWR0114" (id 0) (at 173.99 68.58 0)
+    (property "Reference" "#PWR0115" (id 0) (at 173.99 68.58 0)
       (effects (font (size 1.27 1.27)) hide)
     )
@@
   (symbol (lib_id "power:+5V") (at 242.57 20.32 0) (unit 1)
     (in_bom yes) (on_board yes) (fields_autoplaced)
-    (property "Reference" "#PWR0117" (id 0) (at 242.57 24.13 0)
+    (property "Reference" "#PWR0118" (id 0) (at 242.57 24.13 0)
       (effects (font (size 1.27 1.27)) hide)
     )
@@
   (symbol (lib_id "HC3-rescue:CP") (at 97.79 160.02 0) (unit 1)
     (in_bom yes) (on_board yes)
-    (property "Reference" "C50" (id 0) (at 99.06 157.48 0)
+    (property "Reference" "C58" (id 0) (at 99.06 157.48 0)
       (effects (font (size 1.27 1.27)) (justify left))
     )
@@
   (symbol (lib_id "power:+5V") (at 173.99 19.05 0) (unit 1)
     (in_bom yes) (on_board yes) (fields_autoplaced)
-    (property "Reference" "#PWR0113" (id 0) (at 173.99 22.86 0)
-      (effects (font (size 1.27 1.27)) hide)
-    )
+    (property "Reference" "#PWR0114" (id 0) (at 173.99 22.86 0)
+      (effects (font (size 1.27 1.27)) hide)
+    )

Commit message: Shrink PCB
Parts:
- renumbered J9 to J8
Changed lines of the file:
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@@
   (symbol (lib_id "Connector:Conn_01x02_Male") (at 137.16 175.26 180) (unit 1)
     (in_bom yes) (on_board yes)
-    (property "Reference" "J9" (id 0) (at 137.8712 172.2628 0)
+    (property "Reference" "J8" (id 0) (at 137.8712 172.2628 0)
       (effects (font (size 1.27 1.27)) (justify right))
     )

Commit message: hardware updates
Parts:
- renumbered L11 to L10, L12 to L11, L9 to L8, L10 to L9, R29 to R28, R30 to R29, R31 to R30, R32 to R31, R33 to R32, R34 to R33
Changed lines of the file:
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@@
   (symbol (lib_id "Console-rescue:R") (at 48.26 104.14 270) (unit 1)
     (in_bom yes) (on_board yes)
-    (property "Reference" "R29" (id 0) (at 48.26 106.172 90))
+    (property "Reference" "R28" (id 0) (at 48.26 106.172 90))
     (property "Value" "470kΩ" (id 1) (at 48.26 101.6 90))
     (property "Footprint" "Resistor_THT:R_Axial_DIN0207_L6.3mm_D2.5mm_P7.62mm_Horizontal" (id 2) (at 48.26 102.362 90)
@@
   (symbol (lib_id "Console-rescue:INDUCTANCE_Adjustable_RevE_Date03Aug2010") (at 43.18 96.52 180) (unit 1)
     (in_bom yes) (on_board yes)
-    (property "Reference" "L9" (id 0) (at 43.18 99.06 0)
+    (property "Reference" "L8" (id 0) (at 43.18 99.06 0)
       (effects (font (size 0.762 0.762)))
     )
@@
   (symbol (lib_id "Console-rescue:INDUCTOR_SMALL") (at 107.95 36.83 0) (mirror x) (unit 1)
     (in_bom yes) (on_board yes)
-    (property "Reference" "L12" (id 0) (at 107.95 39.37 0))
+    (property "Reference" "L11" (id 0) (at 107.95 39.37 0))
     (property "Value" "6.8µH" (id 1) (at 107.95 35.56 0))
     (property "Footprint" "Resistor_THT:R_Axial_DIN0207_L6.3mm_D2.5mm_P7.62mm_Horizontal" (id 2) (at 107.95 36.83 0)
@@
   (symbol (lib_id "Console-rescue:R_Small") (at 91.44 45.72 270) (unit 1)
     (in_bom yes) (on_board yes)
-    (property "Reference" "R33" (id 0) (at 91.44 43.18 90))
+    (property "Reference" "R32" (id 0) (at 91.44 43.18 90))
     (property "Value" "470Ω" (id 1) (at 88.9 40.64 90)
       (effects (font (size 1.27 1.27)) (justify left))
@@
   (symbol (lib_id "Console-rescue:INDUCTOR_SMALL") (at 50.8 68.58 90) (unit 1)
     (in_bom yes) (on_board yes)
-    (property "Reference" "L10" (id 0) (at 48.26 68.58 0))
+    (property "Reference" "L9" (id 0) (at 48.26 68.58 0))
     (property "Value" "5.8µH" (id 1) (at 52.07 68.58 0))
     (property "Footprint" "Resistor_THT:R_Axial_DIN0207_L6.3mm_D2.5mm_P7.62mm_Horizontal" (id 2) (at 50.8 68.58 0)
@@
   (symbol (lib_id "HC3-rescue:R") (at 97.79 172.72 90) (unit 1)
     (in_bom yes) (on_board yes)
-    (property "Reference" "R34" (id 0) (at 97.79 170.688 90))
+    (property "Reference" "R33" (id 0) (at 97.79 170.688 90))
     (property "Value" "75Ω" (id 1) (at 97.79 172.72 90))
     (property "Footprint" "Resistor_THT:R_Axial_DIN0207_L6.3mm_D2.5mm_P7.62mm_Horizontal" (id 2) (at 97.79 172.72 0)
@@
   (symbol (lib_id "HC3-rescue:R") (at 48.26 160.02 270) (unit 1)
     (in_bom yes) (on_board yes)
-    (property "Reference" "R30" (id 0) (at 48.26 162.052 90))
+    (property "Reference" "R29" (id 0) (at 48.26 162.052 90))
     (property "Value" "0Ω" (id 1) (at 48.26 160.02 90))
     (property "Footprint" "Resistor_THT:R_Axial_DIN0207_L6.3mm_D2.5mm_P7.62mm_Horizontal" (id 2) (at 48.26 160.02 0)
@@
   (symbol (lib_id "HC3-rescue:R") (at 62.23 166.37 0) (unit 1)
     (in_bom yes) (on_board yes)
-    (property "Reference" "R31" (id 0) (at 64.262 166.37 90))
+    (property "Reference" "R30" (id 0) (at 64.262 166.37 90))
     (property "Value" "470Ω" (id 1) (at 62.23 166.37 90))
     (property "Footprint" "Resistor_THT:R_Axial_DIN0207_L6.3mm_D2.5mm_P7.62mm_Horizontal" (id 2) (at 62.23 166.37 0)
@@
   (symbol (lib_id "HC3-rescue:R") (at 85.09 171.45 0) (unit 1)
     (in_bom yes) (on_board yes)
-    (property "Reference" "R32" (id 0) (at 87.122 171.45 90))
+    (property "Reference" "R31" (id 0) (at 87.122 171.45 90))
     (property "Value" "75Ω" (id 1) (at 85.09 171.45 90))
     (property "Footprint" "Resistor_THT:R_Axial_DIN0207_L6.3mm_D2.5mm_P7.62mm_Horizontal" (id 2) (at 85.09 171.45 0)
@@
   (symbol (lib_id "HC3-rescue:INDUCTOR") (at 97.79 147.32 0) (unit 1)
     (in_bom yes) (on_board yes)
-    (property "Reference" "L11" (id 0) (at 96.52 147.32 90)
+    (property "Reference" "L10" (id 0) (at 96.52 147.32 90)
       (effects (font (size 1.016 1.016)))
     )

Commit message: PCB cleanup
Parts:
- C55, C56, C57: symbol TI-Customs:C_Small -> Device:C
- C58, C60: symbol HC3-rescue:CP -> Device:C_Polarized
- C59: symbol Device:CP -> Device:C_Polarized
- C61: symbol HC3-rescue:C -> Device:C
- L10: symbol HC3-rescue:INDUCTOR -> Device:L_Ferrite
- L11, L9: symbol Console-rescue:INDUCTOR_SMALL -> Device:L
- L8: symbol Console-rescue:INDUCTANCE_Adjustable_RevE_Date03Aug2010 -> Device:L_Trim
- Q2: symbol HC3-rescue:NPN -> Device:Q_NPN_EBC
- R28: symbol Console-rescue:R -> Device:R
- R29, R30, R31, R33: symbol HC3-rescue:R -> Device:R
- R32: symbol Console-rescue:R_Small -> Device:R_Small
- U31: renamed from U30; symbol TI:TMS9918 -> Werner_custom:TMS9918
- Y2: symbol Console-rescue:XTAL_2-TERMINAL_RevE_Date15jun2010 -> Device:Crystal
- renumbered U21 to U22, U31 to U32, U32 to U33, U33 to U34, U34 to U35
Connections:
- net +5V: now also L11.1; no longer L11.2
- net at Y2.1: now also L8.2; no longer L8.1
- net at C55.1, R28.2, U31.40 (XTAL2): now also L8.1; no longer L8.2
- net at C57.1, C59.1, R32.1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: now also L11.2; no longer L11.1
Other:
- moved on the sheet: C55, C56, L11, L8, L9
