File: mainboard/Video.kicad_sch (KiCad schematic)
At the start: 27 parts, among them J8 VIDEO OUT, Q2 2N3904, U22 74LS04, U31 TMS9918, U32 74LS574, U33 74LS574, U34 HM62256BLP, U35 74LS574, U9 74LS32, Y2 10.7MHz

Commit message: PCB rework
Parts:
- removed L11: 6.8µH, Resistor_THT:R_Axial_DIN0207_L6.3mm_D2.5mm_P7.62mm_Horizontal, symbol Device:L
- removed L8: 2- 4.5µH, Resistor_THT:R_Axial_DIN0207_L6.3mm_D2.5mm_P7.62mm_Horizontal, symbol Device:L_Trim
- L7: renamed from L9; footprint Resistor_THT:R_Axial_DIN0207_L6.3mm_D2.5mm_P7.62mm_Horizontal -> Resistor_THT:R_Axial_DIN0207_L6.3mm_D2.5mm_P15.24mm_Horizontal
- renumbered C55 to C56, C56 to C57, C57 to C58, C58 to C59, C59 to C60, C60 to C61, C61 to C62, J8 to J9, L10 to L8, U22 to U24, U31 to U34, U32 to U35, U33 to U36, U34 to U37, U35 to U38
Connections:
- net +5V: now also C58.1, C60.1, R32.1, U34.33 (VCC)
- net at Y2.1: now also C56.1, R28.2, U34.40 (XTAL2)
- net CPUCLK: now reaches U34.38 (CPUCLK)
- no-connect marks 4 -> 3
