File: mainboard/onboardrom.kicad_sch (KiCad schematic)
At the start: 6 parts, among them J17 Rom Select 1, J18 Rom Select 2, SW2 Internal Cart ROM Enable, U43 74LS379, U44 27C010

Commit message: unicorn work
Parts:
- J17, J18: footprint (none) -> Connector_PinSocket_2.54mm:PinSocket_1x03_P2.54mm_Vertical
- R101: footprint (none) -> Resistor_THT:R_Axial_DIN0207_L6.3mm_D2.5mm_P7.62mm_Horizontal
- SW2: footprint (none) -> Connector_PinHeader_2.54mm:PinHeader_1x02_P2.54mm_Vertical
- U43: footprint (none) -> Package_DIP:DIP-16_W7.62mm_Socket_LongPads
- U44: footprint (none) -> Package_DIP:DIP-32_W15.24mm_Socket_LongPads
Changed lines of the file:
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@@
       (effects (font (size 1.27 1.27)) (justify right))
     )
-    (property "Footprint" "" (id 2) (at 176.53 99.06 0)
+    (property "Footprint" "Connector_PinSocket_2.54mm:PinSocket_1x03_P2.54mm_Vertical" (id 2) (at 176.53 99.06 0)
       (effects (font (size 1.27 1.27)) hide)
     )
@@
     (property "Reference" "SW2" (id 0) (at 114.3 54.7202 0))
     (property "Value" "Internal Cart ROM Enable" (id 1) (at 114.3 57.2571 0))
-    (property "Footprint" "" (id 2) (at 114.3 60.96 0)
+    (property "Footprint" "Connector_PinHeader_2.54mm:PinHeader_1x02_P2.54mm_Vertical" (id 2) (at 114.3 60.96 0)
       (effects (font (size 1.27 1.27)) hide)
     )
@@
   (symbol (lib_id "Console-rescue:GND") (at 80.01 147.32 270) (unit 1)
     (in_bom yes) (on_board yes)
-    (property "Reference" "#PWR0190" (id 0) (at 73.66 147.32 0)
+    (property "Reference" "#PWR0191" (id 0) (at 73.66 147.32 0)
       (effects (font (size 1.27 1.27)) hide)
     )
@@
       (effects (font (size 1.27 1.27)) (justify left))
     )
-    (property "Footprint" "" (id 2) (at 53.34 120.65 0)
+    (property "Footprint" "Package_DIP:DIP-16_W7.62mm_Socket_LongPads" (id 2) (at 53.34 120.65 0)
       (effects (font (size 1.27 1.27)) hide)
     )
@@
   (symbol (lib_id "Console-rescue:+5V") (at 53.34 100.33 0) (unit 1)
     (in_bom yes) (on_board yes)
-    (property "Reference" "#PWR0187" (id 0) (at 53.34 104.14 0)
+    (property "Reference" "#PWR0188" (id 0) (at 53.34 104.14 0)
       (effects (font (size 1.27 1.27)) hide)
     )
@@
   (symbol (lib_id "Console-rescue:+5V") (at 78.74 142.24 90) (unit 1)
     (in_bom yes) (on_board yes)
-    (property "Reference" "#PWR0189" (id 0) (at 82.55 142.24 0)
+    (property "Reference" "#PWR0190" (id 0) (at 82.55 142.24 0)
       (effects (font (size 1.27 1.27)) hide)
     )
@@
   (symbol (lib_id "Console-rescue:GND") (at 157.48 116.84 270) (unit 1)
     (in_bom yes) (on_board yes)
-    (property "Reference" "#PWR0195" (id 0) (at 151.13 116.84 0)
+    (property "Reference" "#PWR0196" (id 0) (at 151.13 116.84 0)
       (effects (font (size 1.27 1.27)) hide)
     )
@@
       (effects (font (size 1.27 1.27)) (justify right))
     )
-    (property "Footprint" "" (id 2) (at 177.8 114.3 0)
+    (property "Footprint" "Connector_PinSocket_2.54mm:PinSocket_1x03_P2.54mm_Vertical" (id 2) (at 177.8 114.3 0)
       (effects (font (size 1.27 1.27)) hide)
     )
@@
   (symbol (lib_id "Console-rescue:GND") (at 107.95 160.02 0) (unit 1)
     (in_bom yes) (on_board yes)
-    (property "Reference" "#PWR0192" (id 0) (at 107.95 166.37 0)
+    (property "Reference" "#PWR0193" (id 0) (at 107.95 166.37 0)
       (effects (font (size 1.27 1.27)) hide)
     )
@@
   (symbol (lib_id "Console-rescue:+5V") (at 125.73 44.45 0) (unit 1)
     (in_bom yes) (on_board yes)
-    (property "Reference" "#PWR0193" (id 0) (at 125.73 48.26 0)
+    (property "Reference" "#PWR0194" (id 0) (at 125.73 48.26 0)
       (effects (font (size 1.27 1.27)) hide)
     )
@@
   (symbol (lib_id "Console-rescue:+5V") (at 107.95 86.36 0) (unit 1)
     (in_bom yes) (on_board yes)
-    (property "Reference" "#PWR0191" (id 0) (at 107.95 90.17 0)
+    (property "Reference" "#PWR0192" (id 0) (at 107.95 90.17 0)
       (effects (font (size 1.27 1.27)) hide)
     )
@@
       (effects (font (size 1.27 1.27)) (justify left))
     )
-    (property "Footprint" "" (id 2) (at 123.952 52.07 90)
+    (property "Footprint" "Resistor_THT:R_Axial_DIN0207_L6.3mm_D2.5mm_P7.62mm_Horizontal" (id 2) (at 123.952 52.07 90)
       (effects (font (size 1.27 1.27)) hide)
     )
@@
       (effects (font (size 1.27 1.27)) (justify left))
     )
-    (property "Footprint" "" (id 2) (at 107.95 121.92 0)
+    (property "Footprint" "Package_DIP:DIP-32_W15.24mm_Socket_LongPads" (id 2) (at 107.95 121.92 0)
       (effects (font (size 1.27 1.27)) hide)
     )
@@
   (symbol (lib_id "Console-rescue:GND") (at 53.34 143.51 0) (unit 1)
     (in_bom yes) (on_board yes)
-    (property "Reference" "#PWR0188" (id 0) (at 53.34 149.86 0)
+    (property "Reference" "#PWR0189" (id 0) (at 53.34 149.86 0)
       (effects (font (size 1.27 1.27)) hide)
     )
@@
   (symbol (lib_id "Console-rescue:GND") (at 156.21 101.6 270) (unit 1)
     (in_bom yes) (on_board yes)
-    (property "Reference" "#PWR0194" (id 0) (at 149.86 101.6 0)
-      (effects (font (size 1.27 1.27)) hide)
-    )
+    (property "Reference" "#PWR0195" (id 0) (at 149.86 101.6 0)
+      (effects (font (size 1.27 1.27)) hide)
+    )

Commit message: Shrink PCB
Parts:
- renumbered J17 to J16, J18 to J17
Changed lines of the file:
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@@
   (symbol (lib_id "Connector:Conn_01x03_Male") (at 176.53 99.06 180) (unit 1)
     (in_bom yes) (on_board yes) (fields_autoplaced)
-    (property "Reference" "J17" (id 0) (at 177.2412 98.2253 0)
+    (property "Reference" "J16" (id 0) (at 177.2412 98.2253 0)
       (effects (font (size 1.27 1.27)) (justify right))
     )
@@
   (symbol (lib_id "Connector:Conn_01x03_Male") (at 177.8 114.3 180) (unit 1)
     (in_bom yes) (on_board yes) (fields_autoplaced)
-    (property "Reference" "J18" (id 0) (at 178.5112 113.4653 0)
+    (property "Reference" "J17" (id 0) (at 178.5112 113.4653 0)
       (effects (font (size 1.27 1.27)) (justify right))
     )

Commit message: hardware updates
Parts:
- removed U44: 27C010, Package_DIP:DIP-32_W15.24mm_Socket_LongPads, symbol Memory_EPROM:27C010
- added U44: 27C010-C, Package_DIP:DIP-32_W15.24mm_Socket_LongPads, symbol Werner_custom:27C010-C
- renumbered R101 to R100
Connections:
- net +5V: now also U44.30 (NC), U44.31 (~{PGM}), U44.32 (VCC)
- net A10: now also U44.7 (A5)
- net A11: now also U44.8 (A4)
- net A12: now also U44.9 (A3)
- net A13: now also U44.10 (A2)
- net A15-CRUOUT: now also U44.12 (A0)
- net A3: now also U44.4 (A12)
- net A4: now also U44.25 (A11)
- net A5: now also U44.23 (A10)
- net A6: now also U44.26 (A9)
- net A7: now also U44.27 (A8)
- net A8: now also U44.5 (A7)
- net A9: now also U44.6 (A6)
- net D0: now also U44.21 (D7)
- net D1: now also U44.20 (D6)
- net D2: now also U44.19 (D5)
- net D3: now also U44.18 (D4)
- net D4: now also U44.17 (D3)
- net D5: now also U44.15 (D2)
- net D6: now also U44.14 (D1)
- net D7: now also U44.13 (D0)
- net GND: now also U44.1 (VPP), U44.16 (GND), U44.22 (~{CE})
- net IO_A14: now also U44.11 (A1)
- net IR_A1_O: now also U44.3 (A15)
- net IR_A2_O: now also U44.29 (A14)
- net ~{IROMG}: now also U44.24 (~{OE})
- net at U43.15 (Q3): now also U44.2 (A16)
- net at U43.2 (Q0): now also U44.28 (A13)

Commit message: PCB rework
Parts:
- renumbered R100 to R57, U43 to U44, U44 to U45
Other:
- company: (none) -> Dan Werner - https://github.com/danwerner21/ti99_22
- title: (none) -> TI-99/22
Changed lines of the file:
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@@
 (kicad_sch (version 20211123) (generator eeschema)
   (paper "A4")
+  (title_block
+    (title "TI-99/22")
+    (date "2022-12-26")
+    (rev "0.95")
+    (company "Dan Werner - https://github.com/danwerner21/ti99_22")
+    (comment 1 "Schematic for Keyboard, Joystick and Cassette port.")
+    (comment 3 "was based on the HackMac KiCAD Design")
+    (comment 4 "Based Robert Krenicki's design which")
+    (comment 5 "Original - https://github.com/rkrenicki/TI99-Motherboard")
+  )
   (junction (at 85.09 147.32) (diameter 0) (color 0 0 0 0)
   )
@@
   (symbol (lib_id "power:+5V") (at 121.92 128.27 270) (unit 1)
     (in_bom yes) (on_board yes)
-    (property "Reference" "#PWR0196" (id 0) (at 118.11 128.27 0)
+    (property "Reference" "#PWR0174" (id 0) (at 118.11 128.27 0)
       (effects (font (size 1.27 1.27)) hide)
     )
@@
   (symbol (lib_id "power:GND") (at 80.01 147.32 270) (unit 1)
     (in_bom yes) (on_board yes)
-    (property "Reference" "#PWR0193" (id 0) (at 73.66 147.32 0)
+    (property "Reference" "#PWR0171" (id 0) (at 73.66 147.32 0)
       (effects (font (size 1.27 1.27)) hide)
     )
@@
   (symbol (lib_id "Werner_custom:27C010-C") (at 107.95 121.92 0) (unit 1)
     (in_bom yes) (on_board yes) (fields_autoplaced)
-    (property "Reference" "U44" (id 0) (at 109.9694 90.2802 0)
+    (property "Reference" "U45" (id 0) (at 109.9694 90.2802 0)
       (effects (font (size 1.27 1.27)) (justify left))
     )
@@
   (symbol (lib_id "74xx:74LS379") (at 53.34 120.65 0) (unit 1)
     (in_bom yes) (on_board yes) (fields_autoplaced)
-    (property "Reference" "U43" (id 0) (at 55.3594 104.2502 0)
+    (property "Reference" "U44" (id 0) (at 55.3594 104.2502 0)
       (effects (font (size 1.27 1.27)) (justify left))
     )
@@
   (symbol (lib_id "power:+5V") (at 53.34 100.33 0) (unit 1)
     (in_bom yes) (on_board yes)
-    (property "Reference" "#PWR0190" (id 0) (at 53.34 104.14 0)
+    (property "Reference" "#PWR0168" (id 0) (at 53.34 104.14 0)
       (effects (font (size 1.27 1.27)) hide)
     )
@@
   (symbol (lib_id "power:+5V") (at 78.74 142.24 90) (unit 1)
     (in_bom yes) (on_board yes)
-    (property "Reference" "#PWR0192" (id 0) (at 82.55 142.24 0)
+    (property "Reference" "#PWR0170" (id 0) (at 82.55 142.24 0)
       (effects (font (size 1.27 1.27)) hide)
     )
@@
   (symbol (lib_id "power:GND") (at 157.48 116.84 270) (unit 1)
     (in_bom yes) (on_board yes)
-    (property "Reference" "#PWR0199" (id 0) (at 151.13 116.84 0)
+    (property "Reference" "#PWR0177" (id 0) (at 151.13 116.84 0)
       (effects (font (size 1.27 1.27)) hide)
     )
@@
   (symbol (lib_id "power:GND") (at 107.95 160.02 0) (unit 1)
     (in_bom yes) (on_board yes)
-    (property "Reference" "#PWR0195" (id 0) (at 107.95 166.37 0)
+    (property "Reference" "#PWR0173" (id 0) (at 107.95 166.37 0)
       (effects (font (size 1.27 1.27)) hide)
     )
@@
   (symbol (lib_id "power:+5V") (at 125.73 44.45 0) (unit 1)
     (in_bom yes) (on_board yes)
-    (property "Reference" "#PWR0197" (id 0) (at 125.73 48.26 0)
+    (property "Reference" "#PWR0175" (id 0) (at 125.73 48.26 0)
       (effects (font (size 1.27 1.27)) hide)
     )
@@
   (symbol (lib_id "power:+5V") (at 107.95 86.36 0) (unit 1)
     (in_bom yes) (on_board yes)
-    (property "Reference" "#PWR0194" (id 0) (at 107.95 90.17 0)
+    (property "Reference" "#PWR0172" (id 0) (at 107.95 90.17 0)
       (effects (font (size 1.27 1.27)) hide)
     )
@@
   (symbol (lib_id "Device:R") (at 125.73 52.07 0) (unit 1)
     (in_bom yes) (on_board yes) (fields_autoplaced)
-    (property "Reference" "R100" (id 0) (at 127.508 51.2353 0)
+    (property "Reference" "R57" (id 0) (at 127.508 51.2353 0)
       (effects (font (size 1.27 1.27)) (justify left))
     )
@@
   (symbol (lib_id "power:GND") (at 53.34 143.51 0) (unit 1)
     (in_bom yes) (on_board yes)
-    (property "Reference" "#PWR0191" (id 0) (at 53.34 149.86 0)
+    (property "Reference" "#PWR0169" (id 0) (at 53.34 149.86 0)
       (effects (font (size 1.27 1.27)) hide)
     )
@@
   (symbol (lib_id "power:GND") (at 156.21 101.6 270) (unit 1)
     (in_bom yes) (on_board yes)
-    (property "Reference" "#PWR0198" (id 0) (at 149.86 101.6 0)
-      (effects (font (size 1.27 1.27)) hide)
-    )
+    (property "Reference" "#PWR0176" (id 0) (at 149.86 101.6 0)
+      (effects (font (size 1.27 1.27)) hide)
+    )
